File: Hardware/Amplifiers.sch (KiCad schematic (older format))
At the start: 49 parts, among them U1 TAS5825M

Commit message: Pre refdes fix
Parts:
- C1, C19, C20, C23, C25, C26, C31, C32, C33, C34: renamed from C?; footprint ZOUDIOfootprints:C0805 -> Capacitor_SMD:C_0805_2012Metric
- C10, C15, C16, C17, C18, C2, C3, C4, C7, C9: footprint ZOUDIOfootprints:C0805 -> Capacitor_SMD:C_0805_2012Metric
- C11, C12, C13, C14, C5, C6, C8: footprint ZOUDIOfootprints:C0603 -> Capacitor_SMD:C_0603_1608Metric
- C21, C22, C24, C27, C28, C29, C30: renamed from C?; footprint ZOUDIOfootprints:C0603 -> Capacitor_SMD:C_0603_1608Metric
- J2: renamed from J?; footprint ZOUDIOfootprints:JSTPH_4P -> Connector_JST:JST_PH_B4B-PH-K_1x04_P2.00mm_Vertical
- J3: renamed from J?; footprint ZOUDIOfootprints:PinSocket_1x03_P2.54mm_Vertical -> Connector_JST:JST_PH_B3B-PH-K_1x03_P2.00mm_Vertical
- R7: value 1K -> 1k; footprint ZOUDIOfootprints:R0603 -> Resistor_SMD:R_0603_1608Metric
- gave numbers to parts that had none: 7

Commit message: V0.1 check
Parts:
- removed C29: 470n, Capacitor_SMD:C_0603_1608Metric, symbol Device:C_Small
- added C28: 470n, Capacitor_SMD:C_0603_1608Metric, symbol Device:C_Small
- added C55, C56, C58, C59: 22u, Capacitor_SMD:C_0805_2012Metric, symbol Device:C_Small
- C1: renamed from C35; value 910u -> 820u; footprint ZOUDIOfootprints:Cap_Rad_D10_P5 -> ZOUDIOfootprints:Cap_Rad_D10_P5_horizontal
- C12: renamed from C15; value 470n -> 680n
- C14: renamed from C17; value 470n -> 680n
- C15: renamed from C16; value 470n -> 680n
- C30: renamed from C31; value 470n -> 680n
- C31: renamed from C32; value 470n -> 680n
- C32: renamed from C18; value 470n -> 680n
- C33: value 470n -> 680n
- C40: renamed from C2; value 1u -> 22u
- C41: renamed from C1; value 1u -> 22u
- C43: renamed from C34; value 470n -> 680n
- C52: renamed from C4; value 1u -> 22u
- C53: renamed from C20; value 1u -> 22u
- C57: renamed from C3; value 1u -> 4.7u
- renumbered C13 to C10, C14 to C11, C22 to C18, C6 to C2, C23 to C20, C25 to C24, C26 to C25, C27 to C26, C28 to C27, C30 to C29, C8 to C3, C21 to C38, C24 to C39, C5 to C4, C7 to C5, C9 to C6, C10 to C7, C11 to C8, C12 to C9, J3 to J1, J1 to J4, J2 to J9, L1 to L2, L2 to L3, L3 to L4, L4 to L5, L5 to L6, L6 to L7, L7 to L8, L8 to L9
Connections:
- net GND: now also C55.1, C56.1, C58.1, C59.1
- net VDD: now also C55.2, C56.2, C58.2, C59.2
- net at L8.1, U2.27 (OUT_B-): now also C28.1
- net at U2.28 (BST_B-): now also C28.2
Other:
- moved on the sheet: C1, C10, C11, C12, C14, C15, C18, C19, C2, C20, C24, C25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
