File: Hardware/Bluetooth.sch (KiCad schematic (older format))
At the start: 24 parts, among them J8 U.FL, U4 BTM331

Commit message: Pre refdes fix
Parts:
- C43, C45, C46, C47, C48: footprint ZOUDIOfootprints:C0805 -> Capacitor_SMD:C_0805_2012Metric
- C44: footprint ZOUDIOfootprints:C0603 -> Capacitor_SMD:C_0603_1608Metric
- D2, D3: footprint ZOUDIOfootprints:LED0603 -> LED_SMD:LED_0603_1608Metric
- R12, R13, R14, R15, R16, R17, R18, R19, R20, R21, R22, R23, R24: footprint ZOUDIOfootprints:R0603 -> Resistor_SMD:R_0603_1608Metric
Connections:
- net AUX1_P renamed MIC1_P
- net AUX2_P renamed MIC2_P
- net AUX_N renamed MIC_N
- net USB_N renamed USB_DN
- net USB_P renamed USB_DP
Other:
- moved on the sheet: R13, R14
Changed lines of the file:
@@
 $Descr A4 11693 8268
 encoding utf-8
-Sheet 7 9
+Sheet 8 9
 Title "4x38W amp with DSP and BT"
-Date "2021-05-22"
+Date "2021-06-08"
 Rev "V0.1"
 Comp "ZOUDIO"
@@
 F 0 "R23" H 7400 3550 50  0000 L CNN
 F 1 "10k" H 7350 3450 50  0000 L CNN
-F 2 "ZOUDIOfootprints:R0603" H 7300 3500 50  0001 C CNN
+F 2 "Resistor_SMD:R_0603_1608Metric" H 7300 3500 50  0001 C CNN
 F 3 "~" H 7300 3500 50  0001 C CNN
 F 4 "Uni-royal" H 7300 3500 50  0001 C CNN "Manufacturer"
@@
 F 0 "D3" V 7350 3600 50  0000 C CNN
 F 1 "Blue" V 7250 3600 50  0000 C CNN
-F 2 "ZOUDIOfootprints:LED0603" V 7300 3750 50  0001 C CNN
+F 2 "LED_SMD:LED_0603_1608Metric" V 7300 3750 50  0001 C CNN
 F 3 "~" V 7300 3750 50  0001 C CNN
 F 4 "Orient" H 7300 3750 50  0001 C CNN "Manufacturer"
@@
 F 0 "C45" V 5500 2800 50  0000 C CNN
 F 1 "1u" V 5600 2800 50  0000 C CNN
-F 2 "ZOUDIOfootprints:C0805" H 5550 2700 50  0001 C CNN
+F 2 "Capacitor_SMD:C_0805_2012Metric" H 5550 2700 50  0001 C CNN
 F 3 "~" H 5550 2700 50  0001 C CNN
 F 4 "Yageo" H 5550 2700 50  0001 C CNN "Manufacturer"
@@
 F 0 "C46" V 5500 3350 50  0000 C CNN
 F 1 "1u" V 5600 3350 50  0000 C CNN
-F 2 "ZOUDIOfootprints:C0805" H 5550 3250 50  0001 C CNN
+F 2 "Capacitor_SMD:C_0805_2012Metric" H 5550 3250 50  0001 C CNN
 F 3 "~" H 5550 3250 50  0001 C CNN
 F 4 "Yageo" H 5550 3250 50  0001 C CNN "Manufacturer"
@@
 F 0 "C48" V 5500 3800 50  0000 C CNN
 F 1 "1u" V 5600 3800 50  0000 C CNN
-F 2 "ZOUDIOfootprints:C0805" H 5550 3700 50  0001 C CNN
+F 2 "Capacitor_SMD:C_0805_2012Metric" H 5550 3700 50  0001 C CNN
 F 3 "~" H 5550 3700 50  0001 C CNN
 F 4 "Yageo" H 5550 3700 50  0001 C CNN "Manufacturer"
@@
 F 0 "C44" H 2400 4750 50  0000 C CNN
 F 1 "100n" H 2400 4850 50  0000 C CNN
-F 2 "ZOUDIOfootprints:C0603" H 2550 4750 50  0001 C CNN
+F 2 "Capacitor_SMD:C_0603_1608Metric" H 2550 4750 50  0001 C CNN
 F 3 "~" H 2550 4750 50  0001 C CNN
 F 4 "Walsin" H 2550 4750 50  0001 C CNN "Manufacturer"
@@
 F 0 "R21" V 5900 3200 50  0000 L CNN
 F 1 "1k" V 6000 3200 50  0000 L CNN
-F 2 "ZOUDIOfootprints:R0603" H 6100 3250 50  0001 C CNN
+F 2 "Resistor_SMD:R_0603_1608Metric" H 6100 3250 50  0001 C CNN
 F 3 "~" H 6100 3250 50  0001 C CNN
 F 4 "Uni-royal" H 6100 3250 50  0001 C CNN "Manufacturer"
@@
 F 0 "R18" H 5750 3350 50  0000 L CNN
 F 1 "1k" H 5800 3450 50  0000 L CNN
-F 2 "ZOUDIOfootprints:R0603" H 5950 3400 50  0001 C CNN
+F 2 "Resistor_SMD:R_0603_1608Metric" H 5950 3400 50  0001 C CNN
 F 3 "~" H 5950 3400 50  0001 C CNN
 F 4 "Uni-royal" H 5950 3400 50  0001 C CNN "Manufacturer"
@@
 F 0 "R20" V 5900 2650 50  0000 L CNN
 F 1 "1k" V 6000 2650 50  0000 L CNN
-F 2 "ZOUDIOfootprints:R0603" H 6100 2700 50  0001 C CNN
+F 2 "Resistor_SMD:R_0603_1608Metric" H 6100 2700 50  0001 C CNN
 F 3 "~" H 6100 2700 50  0001 C CNN
 F 4 "Uni-royal" H 6100 2700 50  0001 C CNN "Manufacturer"
@@
 F 0 "R17" H 5750 2800 50  0000 L CNN
 F 1 "1k" H 5800 2900 50  0000 L CNN
-F 2 "ZOUDIOfootprints:R0603" H 5950 2850 50  0001 C CNN
+F 2 "Resistor_SMD:R_0603_1608Metric" H 5950 2850 50  0001 C CNN
 F 3 "~" H 5950 2850 50  0001 C CNN
 F 4 "Uni-royal" H 5950 2850 50  0001 C CNN "Manufacturer"
@@
 F 0 "C43" H 2350 4750 50  0000 C CNN
 F 1 "1u" H 2350 4650 50  0000 C CNN
-F 2 "ZOUDIOfootprints:C0805" H 2200 4750 50  0001 C CNN
+F 2 "Capacitor_SMD:C_0805_2012Metric" H 2200 4750 50  0001 C CNN
 F 3 "~" H 2200 4750 50  0001 C CNN
 F 4 "Yageo" H 2200 4750 50  0001 C CNN "Manufacturer"
@@
 F 0 "R16" H 4250 2550 50  0000 L CNN
 F 1 "0R" H 4300 2650 50  0000 L CNN
-F 2 "ZOUDIOfootprints:R0603" H 4450 2600 50  0001 C CNN
+F 2 "Resistor_SMD:R_0603_1608Metric" H 4450 2600 50  0001 C CNN
 F 3 "~" H 4450 2600 50  0001 C CNN
 F 4 "Uni-royal" H 4450 2600 50  0001 C CNN "Manufacturer"
@@
 F 0 "R19" H 5750 3800 50  0000 L CNN
 F 1 "0R" H 5800 3900 50  0000 L CNN
-F 2 "ZOUDIOfootprints:R0603" H 5950 3850 50  0001 C CNN
+F 2 "Resistor_SMD:R_0603_1608Metric" H 5950 3850 50  0001 C CNN
 F 3 "~" H 5950 3850 50  0001 C CNN
 F 4 "Uni-royal" H 5950 3850 50  0001 C CNN "Manufacturer"
@@
 L power:+5V #PWR0163
 U 1 1 5FC5B431
-P 2300 4200
-F 0 "#PWR0163" H 2300 4050 50  0001 C CNN
-F 1 "+5V" V 2300 4400 50  0000 C CNN
-F 2 "" H 2300 4200 50  0001 C CNN
-F 3 "" H 2300 4200 50  0001 C CNN
-	1    2300 4200
+P 2150 4200
+F 0 "#PWR0163" H 2150 4050 50  0001 C CNN
+F 1 "+5V" V 2150 4400 50  0000 C CNN
+F 2 "" H 2150 4200 50  0001 C CNN
+F 3 "" H 2150 4200 50  0001 C CNN
+	1    2150 4200
 	0    -1   -1   0
 $EndComp
@@
 F 0 "R22" H 7400 2400 50  0000 L CNN
 F 1 "10k" H 7350 2300 50  0000 L CNN
-F 2 "ZOUDIOfootprints:R0603" H 7300 2350 50  0001 C CNN
+F 2 "Resistor_SMD:R_0603_1608Metric" H 7300 2350 50  0001 C CNN
 F 3 "~" H 7300 2350 50  0001 C CNN
 F 4 "Uni-royal" H 7300 2350 50  0001 C CNN "Manufacturer"
@@
 F 0 "D2" V 7350 2450 50  0000 C CNN
 F 1 "Blue" V 7250 2450 50  0000 C CNN
-F 2 "ZOUDIOfootprints:LED0603" V 7300 2600 50  0001 C CNN
+F 2 "LED_SMD:LED_0603_1608Metric" V 7300 2600 50  0001 C CNN
 F 3 "~" V 7300 2600 50  0001 C CNN
 F 4 "Orient" H 7300 2600 50  0001 C CNN "Manufacturer"
@@
 	7300 3350 7300 3400
 Text HLabel 6250 2700 2    50   Input ~ 0
-AUX1_P
+MIC1_P
 Text HLabel 6250 3250 2    50   Input ~ 0
-AUX2_P
+MIC2_P
 Text HLabel 6250 3700 2    50   Input ~ 0
-AUX_N
+MIC_N
 Text HLabel 3150 3400 0    50   Input ~ 0
 PIO19
@@
 L Device:R_Small R13
 U 1 1 5FC19818
-P 2500 4200
-F 0 "R13" V 2400 4050 50  0000 L CNN
-F 1 "0R" V 2400 4250 50  0000 L CNN
-F 2 "ZOUDIOfootprints:R0603" H 2500 4200 50  0001 C CNN
-F 3 "~" H 2500 4200 50  0001 C CNN
-F 4 "Uni-royal" H 2500 4200 50  0001 C CNN "Manufacturer"
-F 5 "0603WAF0000T5E" H 2500 4200 50  0001 C CNN "Partnumber"
-	1    2500 4200
-	0    1    1    0
-$EndComp
-Wire Wire Line
-	2300 4200 2350 4200
+P 2350 4200
+F 0 "R13" V 2250 4050 50  0000 L CNN
+F 1 "0R" V 2250 4250 50  0000 L CNN
+F 2 "Resistor_SMD:R_0603_1608Metric" H 2350 4200 50  0001 C CNN
+F 3 "~" H 2350 4200 50  0001 C CNN
+F 4 "Uni-royal" H 2350 4200 50  0001 C CNN "Manufacturer"
+F 5 "0603WAF0000T5E" H 2350 4200 50  0001 C CNN "Partnumber"
+	1    2350 4200
+	0    1    1    0
+$EndComp
+Wire Wire Line
+	2150 4200 2200 4200
 $Comp
 L Device:R_Small R?
@@
 F 0 "R12" H 2259 5546 50  0000 L CNN
 F 1 "10k" H 2259 5455 50  0000 L CNN
-F 2 "ZOUDIOfootprints:R0603" H 2200 5500 50  0001 C CNN
+F 2 "Resistor_SMD:R_0603_1608Metric" H 2200 5500 50  0001 C CNN
 F 3 "~" H 2200 5500 50  0001 C CNN
 F 4 "Uni-royal" H 2200 5500 50  0001 C CNN "Manufacturer"
@@
 F 0 "R15" H 2609 5546 50  0000 L CNN
 F 1 "10k" H 2609 5455 50  0000 L CNN
-F 2 "ZOUDIOfootprints:R0603" H 2550 5500 50  0001 C CNN
+F 2 "Resistor_SMD:R_0603_1608Metric" H 2550 5500 50  0001 C CNN
 F 3 "~" H 2550 5500 50  0001 C CNN
 F 4 "Uni-royal" H 2550 5500 50  0001 C CNN "Manufacturer"
@@
 	2200 5650 2200 5600
 Wire Wire Line
-	2400 4300 2350 4300
-Wire Wire Line
-	2350 4300 2350 4200
-Connection ~ 2350 4200
-Wire Wire Line
-	2350 4200 2400 4200
+	2250 4300 2200 4300
+Wire Wire Line
+	2200 4300 2200 4200
+Connection ~ 2200 4200
+Wire Wire Line
+	2200 4200 2250 4200
 $Comp
 L Device:R_Small R?
@@
 F 0 "R24" V 2800 4400 50  0000 C CNN
 F 1 "10k" V 2800 4600 50  0000 C CNN
-F 2 "ZOUDIOfootprints:R0603" H 2900 4500 50  0001 C CNN
+F 2 "Resistor_SMD:R_0603_1608Metric" H 2900 4500 50  0001 C CNN
 F 3 "~" H 2900 4500 50  0001 C CNN
 F 4 "Uni-royal" H 2900 4500 50  0001 C CNN "Manufacturer"
@@
 Wire Wire Line
 	2800 4500 2750 4500
-Text HLabel 2750 4500 0    50   Input ~ 0
-Enable
 Text HLabel 4350 5100 3    50   Input ~ 0
 PIO4
@@
 Text Notes 1700 1950 0    50   ~ 0
 Bluetooth module
-Wire Wire Line
-	2600 4300 3150 4300
-Wire Wire Line
-	2600 4200 3150 4200
 $Comp
 L Device:R_Small R14
 U 1 1 5FD0344A
-P 2500 4300
-F 0 "R14" V 2600 4150 50  0000 L CNN
-F 1 "0R" V 2600 4350 50  0000 L CNN
-F 2 "ZOUDIOfootprints:R0603" H 2500 4300 50  0001 C CNN
-F 3 "~" H 2500 4300 50  0001 C CNN
-F 4 "Uni-royal" H 2500 4300 50  0001 C CNN "Manufacturer"
-F 5 "0603WAF0000T5E" H 2500 4300 50  0001 C CNN "Partnumber"
-	1    2500 4300
+P 2350 4300
+F 0 "R14" V 2450 4150 50  0000 L CNN
+F 1 "0R" V 2450 4350 50  0000 L CNN
+F 2 "Resistor_SMD:R_0603_1608Metric" H 2350 4300 50  0001 C CNN
+F 3 "~" H 2350 4300 50  0001 C CNN
+F 4 "Uni-royal" H 2350 4300 50  0001 C CNN "Manufacturer"
+F 5 "0603WAF0000T5E" H 2350 4300 50  0001 C CNN "Partnumber"
+	1    2350 4300
 	0    1    1    0
 $EndComp
@@
 F 0 "C47" V 5500 3600 50  0000 C CNN
 F 1 "1u" V 5600 3600 50  0000 C CNN
-F 2 "ZOUDIOfootprints:C0805" H 5550 3500 50  0001 C CNN
+F 2 "Capacitor_SMD:C_0805_2012Metric" H 5550 3500 50  0001 C CNN
 F 3 "~" H 5550 3500 50  0001 C CNN
 F 4 "Yageo" H 5550 3500 50  0001 C CNN "Manufacturer"
@@
 DNP R16 to use \nU.FL connector
 Text HLabel 3150 4000 0    50   BiDi ~ 0
-USB_N
+USB_DN
 Text HLabel 3150 4100 0    50   BiDi ~ 0
-USB_P
+USB_DP
 NoConn ~ 4550 5100
+Text HLabel 2750 4500 0    50   Input ~ 0
+Enable
+Wire Wire Line
+	2450 4300 3150 4300
+Wire Wire Line
+	2450 4200 3150 4200
 $EndSCHEMATC

Commit message: V0.1 check
Parts:
- added J11: JST-PH 01x02, Connector_JST:JST_PH_B2B-PH-K_1x02_P2.00mm_Vertical, symbol Connector_Generic:Conn_01x02
- added R42: 1k, Resistor_SMD:R_0603_1608Metric, symbol Device:R_Small
- renumbered C43 to C45, C44 to C46, C45 to C48, C46 to C49, C47 to C50, C48 to C51, D2 to D6, D3 to D7, J8 to J10, R12 to R29, R13 to R30, R14 to R31, R15 to R32, R24 to R33, R16 to R34, R17 to R35, R18 to R36, R19 to R37, R20 to R38, R21 to R39, R22 to R40, R23 to R41, U4 to U10
Connections:
- net +3V3: now also R42.1
- net LED5: now also J11.2 (Pin_2)
- net +5V renamed 5V_usb
- net PIO23: no longer names the net of U10.51 (PIO23)
- new net: J11.1 (Pin_1), R42.2
- no-connect marks 21 -> 22
Other:
- note added: "Default input is single-ended\nDNP R37 for differential input"
- note removed: "Default input is single-ended\nDNP R20 for differential input"
- moved on the sheet: D7, R41
