File: Hardware/Power.sch (KiCad schematic (older format))
At the start: 12 parts, among them Q2 P-Channel, U3 TPS62177

Commit message: Pre refdes fix
Parts:
- removed C41, C42: 10u, ZOUDIOfootprints:C1206, symbol Device:C
- removed U3: TPS62177, ZOUDIOfootprints:WSON10EP, symbol ZOUDIOsymbols:TPS62177
- added C38, C41: 10u, Capacitor_SMD:C_0805_2012Metric, symbol Device:C_Small
- added C39, C40: 100n, Capacitor_SMD:C_0603_1608Metric, symbol Device:C_Small
- added R35, R36: 100k, Resistor_SMD:R_0603_1608Metric, symbol Device:R_Small
- added R37: 500R, Resistor_SMD:R_0603_1608Metric, symbol Device:R_Small
- added U11: TPS2113A, Package_SO:TSSOP-8_3x3mm_P0.65mm, symbol ZOUDIOsymbols:TPS2113A
- added U3: TLV1117-33, Package_TO_SOT_SMD:SOT-23, symbol Regulator_Linear:TLV1117-33
- added U7: TPS62177DQC, Package_SON:WSON-10-1EP_2x3mm_P0.5mm_EP0.84x2.4mm_ThermalVias, symbol Regulator_Switching:TPS62177DQC
- C36, C37: footprint ZOUDIOfootprints:C0805 -> Capacitor_SMD:C_0805_2012Metric
- D1: footprint ZOUDIOfootprints:D_SMA -> Diode_SMD:D_SMA
- R10, R8: footprint ZOUDIOfootprints:R0603 -> Resistor_SMD:R_0603_1608Metric
- R11, R9: value 100K -> 100k; footprint ZOUDIOfootprints:R0603 -> Resistor_SMD:R_0603_1608Metric
Connections:
- net +3V3: now also U11.7 (OUT); no longer L9.2
- net Buck_sleep: now also U7.8 (~SLEEP)
- net GND: now also C38.2, C39.2, C40.1, C41.2, R36.1, R37.2, U11.2 (/EN), U11.5 (GND), U3.1 (GND), U7.1 (PGND), U7.11 (PAD), U7.4 (NC), U7.5 (FB), U7.6 (AGND)
- net VDD: now also U7.2 (VIN), U7.3 (EN)
- net at L9.1: now also U7.9 (SW)
- new net: R35.1, R36.2, U11.3 (VSNS)
- new net: R37.1, U11.4 (ILIM)
- new net +5V: C39.1, U3.3 (VI)
- new net 3V3_buck: C38.1, C41.1, L9.2, U11.6 (IN2), U7.10 (VOS)
- new net 3V3_ldo: C40.2, R35.2, U11.8 (IN1), U3.2 (VO)
- no-connect marks 1 -> 2
Other:
- note added: "3V3 LDO"
- note added: "3V3 multiplexer"
- moved on the sheet: C36, C37, D1, L9, Q2, R10, R11, R8, R9

Commit message: V0.1 check
Parts:
- removed C39, C40: 100n, Capacitor_SMD:C_0603_1608Metric, symbol Device:C_Small
- removed U3: TLV1117-33, Package_TO_SOT_SMD:SOT-23, symbol Regulator_Linear:TLV1117-33
- added C13, C16: 1u, Capacitor_SMD:C_0805_2012Metric, symbol Device:C_Small
- added R43: 525k, Resistor_SMD:R_0603_1608Metric, symbol Device:R_Small
- added R44: 100k, Resistor_SMD:R_0603_1608Metric, symbol Device:R_Small
- added U11: LP5907MFX-3.3, Package_TO_SOT_SMD:SOT-23-5, symbol Regulator_Linear:LP5907MFX-3.3
- R10: renamed from R37; value 500R -> 1K
- R8: renamed from R35; value 100k -> 10k
- U4: renamed from U7; value TPS62177DQC -> TPS62175DQC; symbol Regulator_Switching:TPS62177DQC -> Regulator_Switching:TPS62175DQC
- renumbered C36 to C21, C37 to C22, C38 to C23, C41 to C47, D1 to D2, L9 to L1, Q2 to Q1, R10 to R1, R11 to R3, R8 to R5, R9 to R6, R36 to R9, U11 to U5
Connections:
- net 3V3_ldo is gone; now on net 5V_buck: R8.2, U5.8 (IN1)
- net +3V3: now also C16.1, U11.5 (OUT); no longer U5.7 (OUT)
- net +5V: now also U5.7 (OUT), C13.1, U11.1 (IN), U11.3 (EN)
- net GND: now also C13.2, C16.2, R44.2, U11.2 (GND); no longer U4.5 (FB)
- net 3V3_buck renamed 5V_buck
- net 5V_buck: now also R43.1; no longer U5.6 (IN2)
- new net: R43.2, R44.1, U4.5 (FB)
- new net 5V_usb: U5.6 (IN2)
Other:
- note added: "3.3V LDO"
- note added: "5V buckconverter"
- note added: "5V multiplexer"
- note added: "ERC"
- note added: "If VSNS < 0.8V (5V_buck < 4.55V) IN2 is selected"
- note added: "Ilim = 500/R10 = 0.5A"
- note removed: "3V3 LDO"
- note removed: "3V3 buckconverter"
- note removed: "3V3 multiplexer"
- moved on the sheet: C21, C22, D2, L1, Q1, R1, R10, R3, R5, R6, R8, R9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
