File: Hardware/USB to UART.sch (KiCad schematic (older format))
At the start: 8 parts, among them U7 CH340C

Commit message: Pre refdes fix
Parts:
- removed U7: CH340C, ZOUDIOfootprints:SOIC-16_3.9x9.9mm_P1.27mm, symbol ZOUDIOsymbols:CH340C
- added U10: CH340C, Package_SO:SOIC-16_3.9x9.9mm_P1.27mm, symbol Interface_USB:CH340C
- C51: footprint ZOUDIOfootprints:C0603 -> Capacitor_SMD:C_0603_1608Metric
- D4, D5, D6: footprint ZOUDIOfootprints:LED0603 -> LED_SMD:LED_0603_1608Metric
- R32, R33, R34: footprint ZOUDIOfootprints:R0603 -> Resistor_SMD:R_0603_1608Metric
Connections:
- net +3V3: now also U10.16 (VCC), U10.4 (V3)
- net GND: now also U10.1 (GND)
- net UART_DTR: now also U10.13 (~DTR)
- net UART_RX: now also U10.3 (RXD)
- net UART_TX: now also U10.2 (TXD)
- new net UD+: U10.5 (UD+)
- new net UD-: U10.6 (UD-)
- no-connect marks 8 -> 6
Other:
- note added: "TODO: switch to -B"
- moved on the sheet: C51
Changed lines of the file:
@@
 $Descr A4 11693 8268
 encoding utf-8
-Sheet 2 9
+Sheet 7 9
 Title "4x38W amp with DSP and BT"
-Date "2021-05-22"
+Date "2021-06-08"
 Rev "V0.1"
 Comp "ZOUDIO"
@@
 $EndDescr
 $Comp
-L ZOUDIOsymbols:CH340C U?
-U 1 1 5FD85CD8
-P 4650 3500
-AR Path="/5FD85CD8" Ref="U?"  Part="1"
-AR Path="/5FD15AD6/5FD85CD8" Ref="U?"  Part="1"
-AR Path="/5FBDE62F/5FD85CD8" Ref="U?"  Part="1"
-AR Path="/5FD81784/5FD85CD8" Ref="U?"  Part="1"
-AR Path="/5FCDB1AE/5FD85CD8" Ref="U?"  Part="1"
-AR Path="/5FF9E05B/5FD85CD8" Ref="U?"  Part="1"
-AR Path="/60A7E145/5FD85CD8" Ref="U7"  Part="1"
-F 0 "U7" H 4650 4075 50  0000 C CNN
-F 1 "CH340C" H 4650 3984 50  0000 C CNN
-F 2 "ZOUDIOfootprints:SOIC-16_3.9x9.9mm_P1.27mm" H 4400 3750 50  0001 C CNN
-F 3 "" H 4400 3750 50  0001 C CNN
-F 4 "WCH" H 4650 3500 50  0001 C CNN "Manufacturer"
-F 5 "CH340C" H 4650 3500 50  0001 C CNN "Partnumber"
-	1    4650 3500
-	1    0    0    -1
-$EndComp
-$Comp
 L power:GND #PWR?
 U 1 1 5FD85CDF
-P 4250 3150
+P 4800 4450
 AR Path="/5FD85CDF" Ref="#PWR?"  Part="1"
 AR Path="/5FD15AD6/5FD85CDF" Ref="#PWR?"  Part="1"
@@
 AR Path="/5FF9E05B/5FD85CDF" Ref="#PWR?"  Part="1"
 AR Path="/60A7E145/5FD85CDF" Ref="#PWR0187"  Part="1"
-F 0 "#PWR0187" H 4250 2900 50  0001 C CNN
-F 1 "GND" H 4255 2977 50  0001 C CNN
-F 2 "" H 4250 3150 50  0001 C CNN
-F 3 "" H 4250 3150 50  0001 C CNN
-	1    4250 3150
-	0    1    1    0
-$EndComp
-Wire Wire Line
-	4300 3150 4250 3150
-NoConn ~ 4300 3850
-NoConn ~ 4300 3750
+F 0 "#PWR0187" H 4800 4200 50  0001 C CNN
+F 1 "GND" H 4805 4277 50  0001 C CNN
+F 2 "" H 4800 4450 50  0001 C CNN
+F 3 "" H 4800 4450 50  0001 C CNN
+	1    4800 4450
+	1    0    0    -1
+$EndComp
 $Comp
 L Device:R_Small R?
@@
 F 0 "R34" H 6500 5100 50  0000 L CNN
 F 1 "10k" H 6500 5000 50  0000 L CNN
-F 2 "ZOUDIOfootprints:R0603" H 6450 5050 50  0001 C CNN
+F 2 "Resistor_SMD:R_0603_1608Metric" H 6450 5050 50  0001 C CNN
 F 3 "~" H 6450 5050 50  0001 C CNN
 F 4 "Uni-royal" H 6450 5050 50  0001 C CNN "Manufacturer"
@@
 F 0 "D6" V 6500 5150 50  0000 C CNN
 F 1 "Blue" V 6400 5150 50  0000 C CNN
-F 2 "ZOUDIOfootprints:LED0603" V 6450 5300 50  0001 C CNN
+F 2 "LED_SMD:LED_0603_1608Metric" V 6450 5300 50  0001 C CNN
 F 3 "~" V 6450 5300 50  0001 C CNN
 F 4 "Orient" H 6450 5300 50  0001 C CNN "Manufacturer"
@@
 F 0 "R33" H 6500 4200 50  0000 L CNN
 F 1 "10k" H 6500 4100 50  0000 L CNN
-F 2 "ZOUDIOfootprints:R0603" H 6450 4150 50  0001 C CNN
+F 2 "Resistor_SMD:R_0603_1608Metric" H 6450 4150 50  0001 C CNN
 F 3 "~" H 6450 4150 50  0001 C CNN
 F 4 "Uni-royal" H 6450 4150 50  0001 C CNN "Manufacturer"
@@
 F 0 "D5" V 6500 4250 50  0000 C CNN
 F 1 "Blue" V 6400 4250 50  0000 C CNN
-F 2 "ZOUDIOfootprints:LED0603" V 6450 4400 50  0001 C CNN
+F 2 "LED_SMD:LED_0603_1608Metric" V 6450 4400 50  0001 C CNN
 F 3 "~" V 6450 4400 50  0001 C CNN
 F 4 "Orient" H 6450 4400 50  0001 C CNN "Manufacturer"
@@
 F 0 "R32" H 6500 3250 50  0000 L CNN
 F 1 "10k" H 6500 3150 50  0000 L CNN
-F 2 "ZOUDIOfootprints:R0603" H 6450 3200 50  0001 C CNN
+F 2 "Resistor_SMD:R_0603_1608Metric" H 6450 3200 50  0001 C CNN
 F 3 "~" H 6450 3200 50  0001 C CNN
 F 4 "Uni-royal" H 6450 3200 50  0001 C CNN "Manufacturer"
@@
 F 0 "D4" V 6500 3300 50  0000 C CNN
 F 1 "Blue" V 6400 3300 50  0000 C CNN
-F 2 "ZOUDIOfootprints:LED0603" V 6450 3450 50  0001 C CNN
+F 2 "LED_SMD:LED_0603_1608Metric" V 6450 3450 50  0001 C CNN
 F 3 "~" V 6450 3450 50  0001 C CNN
 F 4 "Orient" H 6450 3450 50  0001 C CNN "Manufacturer"
@@
 Wire Wire Line
 	6450 3650 6400 3650
-NoConn ~ 5000 3550
-NoConn ~ 5000 3650
-NoConn ~ 5000 3750
-NoConn ~ 5000 3850
-NoConn ~ 5000 3250
 $Comp
 L power:+3V3 #PWR?
 U 1 1 5FD85D3A
-P 5050 3100
+P 4800 3050
 AR Path="/5FD85D3A" Ref="#PWR?"  Part="1"
 AR Path="/5FCC1D27/5FD85D3A" Ref="#PWR?"  Part="1"
@@
 AR Path="/5FF9E05B/5FD85D3A" Ref="#PWR?"  Part="1"
 AR Path="/60A7E145/5FD85D3A" Ref="#PWR0189"  Part="1"
-F 0 "#PWR0189" H 5050 2950 50  0001 C CNN
-F 1 "+3V3" H 5065 3273 50  0000 C CNN
-F 2 "" H 5050 3100 50  0001 C CNN
-F 3 "" H 5050 3100 50  0001 C CNN
-	1    5050 3100
+F 0 "#PWR0189" H 4800 2900 50  0001 C CNN
+F 1 "+3V3" H 4815 3223 50  0000 C CNN
+F 2 "" H 4800 3050 50  0001 C CNN
+F 3 "" H 4800 3050 50  0001 C CNN
+	1    4800 3050
 	1    0    0    -1
 $EndComp
@@
 L power:GND #PWR?
 U 1 1 5FD85D4B
-P 5450 3150
+P 5200 3100
 AR Path="/5FD85D4B" Ref="#PWR?"  Part="1"
 AR Path="/5FD15AD6/5FD85D4B" Ref="#PWR?"  Part="1"
@@
 AR Path="/5FF9E05B/5FD85D4B" Ref="#PWR?"  Part="1"
 AR Path="/60A7E145/5FD85D4B" Ref="#PWR0190"  Part="1"
-F 0 "#PWR0190" H 5450 2900 50  0001 C CNN
-F 1 "GND" H 5455 2977 50  0001 C CNN
-F 2 "" H 5450 3150 50  0001 C CNN
-F 3 "" H 5450 3150 50  0001 C CNN
-	1    5450 3150
+F 0 "#PWR0190" H 5200 2850 50  0001 C CNN
+F 1 "GND" H 5205 2927 50  0001 C CNN
+F 2 "" H 5200 3100 50  0001 C CNN
+F 3 "" H 5200 3100 50  0001 C CNN
+	1    5200 3100
 	0    -1   -1   0
 $EndComp
-$Comp
-L power:+3V3 #PWR?
-U 1 1 5FD85D52
-P 4250 3450
-AR Path="/5FD85D52" Ref="#PWR?"  Part="1"
-AR Path="/5FCC1D27/5FD85D52" Ref="#PWR?"  Part="1"
-AR Path="/5FBDE62F/5FD85D52" Ref="#PWR?"  Part="1"
-AR Path="/5FD81784/5FD85D52" Ref="#PWR?"  Part="1"
-AR Path="/5FCDB1AE/5FD85D52" Ref="#PWR?"  Part="1"
-AR Path="/5FF9E05B/5FD85D52" Ref="#PWR?"  Part="1"
-AR Path="/60A7E145/5FD85D52" Ref="#PWR0191"  Part="1"
-F 0 "#PWR0191" H 4250 3300 50  0001 C CNN
-F 1 "+3V3" V 4250 3700 50  0000 C CNN
-F 2 "" H 4250 3450 50  0001 C CNN
-F 3 "" H 4250 3450 50  0001 C CNN
-	1    4250 3450
-	0    -1   -1   0
-$EndComp
-Wire Wire Line
-	4300 3450 4250 3450
-NoConn ~ 5000 3350
-Text HLabel 4300 3250 0    50   Output ~ 0
+Text HLabel 5200 3400 2    50   Output ~ 0
 UART_TX
-Text HLabel 4300 3350 0    50   Input ~ 0
+Text HLabel 5200 3500 2    50   Input ~ 0
 UART_RX
-Text HLabel 5000 3450 2    50   Output ~ 0
+Text HLabel 5200 4100 2    50   Output ~ 0
 UART_DTR
 Text Notes 6800 3350 0    50   ~ 0
@@
 UART_TX LOW = Bit outgoing
 Wire Notes Line
-	3800 2800 5650 2800
-Wire Notes Line
-	5650 2800 5650 4050
-Wire Notes Line
-	5650 4050 3800 4050
-Wire Notes Line
-	3800 4050 3800 2800
-Text Notes 3800 2800 0    50   ~ 0
+	4000 2800 5650 2800
+Wire Notes Line
+	5650 2800 5650 4750
+Wire Notes Line
+	5650 4750 4000 4750
+Wire Notes Line
+	4000 4750 4000 2800
+Text Notes 4000 2800 0    50   ~ 0
 USB to UART converter
 Text HLabel 6400 4550 0    50   Input ~ 0
@@
 	1    0    0    -1
 $EndComp
-Text HLabel 4300 3550 0    50   BiDi ~ 0
-USB_D+
-Text HLabel 4300 3650 0    50   BiDi ~ 0
-USB_D-
+Text HLabel 4400 3700 0    50   BiDi ~ 0
+UD+
+Text HLabel 4400 3800 0    50   BiDi ~ 0
+UD-
 Text HLabel 6400 3650 0    50   Output ~ 0
 UART_DTR
-Wire Wire Line
-	5000 3150 5050 3150
-Wire Wire Line
-	5050 3100 5050 3150
 $Comp
 L Device:C_Small C?
 U 1 1 5FD85D40
-P 5200 3150
+P 4950 3100
 AR Path="/5FD85D40" Ref="C?"  Part="1"
 AR Path="/5FCC1D27/5FD85D40" Ref="C?"  Part="1"
@@
 AR Path="/5FF9E05B/5FD85D40" Ref="C?"  Part="1"
 AR Path="/60A7E145/5FD85D40" Ref="C51"  Part="1"
-F 0 "C51" V 5150 3300 50  0000 C CNN
-F 1 "100n" V 5250 3300 50  0000 C CNN
-F 2 "ZOUDIOfootprints:C0603" H 5200 3150 50  0001 C CNN
-F 3 "~" H 5200 3150 50  0001 C CNN
-F 4 "Walsin" H 5200 3150 50  0001 C CNN "Manufacturer"
-F 5 "0603B104J500CT" H 5200 3150 50  0001 C CNN "Partnumber"
-	1    5200 3150
+F 0 "C51" V 4900 3250 50  0000 C CNN
+F 1 "100n" V 5000 3250 50  0000 C CNN
+F 2 "Capacitor_SMD:C_0603_1608Metric" H 4950 3100 50  0001 C CNN
+F 3 "~" H 4950 3100 50  0001 C CNN
+F 4 "Walsin" H 4950 3100 50  0001 C CNN "Manufacturer"
+F 5 "0603B104J500CT" H 4950 3100 50  0001 C CNN "Partnumber"
+	1    4950 3100
 	0    1    1    0
 $EndComp
 Wire Wire Line
-	5450 3150 5300 3150
-Wire Wire Line
-	5100 3150 5050 3150
-Connection ~ 5050 3150
+	5200 3100 5050 3100
+Wire Wire Line
+	4850 3100 4800 3100
 Wire Notes Line
 	5900 2800 8050 2800
@@
 Wire Notes Line
 	5900 5550 8050 5550
+Wire Wire Line
+	4800 3050 4800 3100
+Wire Wire Line
+	4700 3200 4700 3100
+Wire Wire Line
+	4700 3100 4800 3100
+Connection ~ 4800 3100
+Wire Wire Line
+	4800 3100 4800 3200
+NoConn ~ 4400 3500
+NoConn ~ 5200 3700
+NoConn ~ 5200 3800
+NoConn ~ 5200 3900
+NoConn ~ 5200 4000
+NoConn ~ 5200 4200
+Wire Wire Line
+	4800 4400 4800 4450
+$Comp
+L Interface_USB:CH340C U10
+U 1 1 60B2C7AB
+P 4800 3800
+F 0 "U10" H 4550 4350 50  0000 C CNN
+F 1 "CH340C" H 5000 4350 50  0000 C CNN
+F 2 "Package_SO:SOIC-16_3.9x9.9mm_P1.27mm" H 4850 3250 50  0001 L CNN
+F 3 "https://datasheet.lcsc.com/szlcsc/Jiangsu-Qin-Heng-CH340C_C84681.pdf" H 4450 4600 50  0001 C CNN
+	1    4800 3800
+	1    0    0    -1
+$EndComp
+Text Notes 3400 4400 0    50   ~ 0
+TODO: switch to -B
 $EndSCHEMATC

Commit message: V0.1 check
Parts:
- U9: renamed from U10; value CH340C -> CH340B
- renumbered C51 to C44, D4 to D3, D5 to D4, D6 to D5, R32 to R26, R33 to R27, R34 to R28
Connections:
- net +3V3 renamed VCC
Other:
- note added: "Note:\nPincompatible with CH340C,\nwhich has no configurable VID/PID"
- note removed: "TODO: switch to -B"
- moved on the sheet: D3, D4, D5, R26, R27, R28
