File: Hardware/USB.sch (KiCad schematic (older format))
At the start: 4 parts

Commit message: Pre refdes fix
Parts:
- removed Y?: 12Mhz, symbol Device:Crystal_GND23_Small
- added C53, C54, C55: 10u, Capacitor_SMD:C_0805_2012Metric, symbol Device:C_Small
- added D7: Blue, LED_SMD:LED_0603_1608Metric, symbol Device:LED_Small
- added F1: 500mA, symbol Device:Polyfuse_Small
- added FB1, FB2, FB3, FB4, FB5: 120R, Capacitor_SMD:C_0603_1608Metric, symbol Device:Ferrite_Bead_Small
- added R38, R41: 100k, Resistor_SMD:R_0603_1608Metric, symbol Device:R_Small
- added R39: 10k, Resistor_SMD:R_0603_1608Metric, symbol Device:R_Small
- added R40: 47k, Resistor_SMD:R_0603_1608Metric, symbol Device:R_Small
- added R6: 1k, Resistor_SMD:R_0603_1608Metric, symbol Device:R_Small
- added TP1, TP2, TP3, TP4, TP5: TestPoint, TestPoint:TestPoint_Pad_D1.0mm, symbol Connector:TestPoint
- added Y1: 12MHz, Crystal:Crystal_SMD_Abracon_ABM3C-4Pin_5.0x3.2mm, symbol Device:Crystal_GND23_Small
- J4: renamed from J?; footprint (none) -> Connector_USB:USB_Micro-B_Molex-105017-0001; Function (none) -> Hub input
- R1: renamed from R?; value 10k -> 2k7; footprint (none) -> Resistor_SMD:R_0603_1608Metric
- gave numbers to parts that had none: 1
Connections:
- net +5V: now also U8.20 (VDD5), C55.2, F1.1, R38.1, R40.1; no longer J4.1 (VBUS), U8.18 (VBUSM)
- net DM1: now also FB2.1; no longer U8.10 (DM1)
- net DM2: now also FB4.1; no longer U8.8 (DM2)
- net DP1: now also FB1.1; no longer U8.11 (DP1)
- net DP2: now also FB3.1; no longer U8.9 (DP2)
- net GND: now also C53.1, C54.1, C55.1, FB5.1, R39.1, R41.2, R6.2, Y1.2, Y1.3; no longer J4.6 (Shield), U8.27 (TESTJ/EESDA)
- net 1V8: now reaches U8.12 (VD18_O)
- net 1V8: now also U8.28 (VD18), C54.2
- net 3V3: now reaches U8.13 (VD33)
- net 3V3: now also U8.21 (VD33_O), C53.2
- net at U8.17 (~XRSTJ): now also R38.2
- net at U8.19 (BUSJ): now also R39.2
- net at U8.2 (XOUT): now also Y1.1
- net DRV: now reaches U8.22 (DRV)
- net DRV: now also D7.2 (A)
- net I2C_SCL: now reaches U8.23 (LED1/EESCL)
- net I2C_SCL: now also TP1.1, TP3.1
- net LED2: now reaches U8.24 (LED2)
- net LED2: now also TP4.1
- net OVCJ: now reaches U8.26 (OVCJ)
- net OVCJ: now also TP5.1
- net at U8.3 (XIN): now also Y1.4
- net USB_D+: no longer names the net of J4.3 (D+), U8.16 (DPU)
- net USB_D-: no longer names the net of J4.2 (D-), U8.15 (DMU)
- new net: R40.2, R41.1, U8.18 (VBUSM)
- new net: FB2.2, U8.10 (DM1)
- new net: FB1.2, U8.11 (DP1)
- new net: FB4.2, U8.8 (DM2)
- new net: FB3.2, U8.9 (DP2)
- new net: F1.2, J4.1 (VBUS)
- new net: D7.1 (K), R6.1
- new net: FB5.2, J4.6 (Shield)
- new net I2C_SDA: TP2.1, U8.27 (TESTJ/EESDA)
- no-connect marks 8 -> 6
Other:
- note added: "Hub active led"
- note added: "Testpoints"
- note added: "USB hub controller"
- note removed: "Todo: finish USB 2-port hub IC circuit"
- moved on the sheet: J4, R1, U8

Commit message: V0.1 check
Parts:
- removed C53, C54: 10u, Capacitor_SMD:C_0805_2012Metric, symbol Device:C_Small
- removed R40: 47k, Resistor_SMD:R_0603_1608Metric, symbol Device:R_Small
- removed R41: 100k, Resistor_SMD:R_0603_1608Metric, symbol Device:R_Small
- removed TP3, TP5: TestPoint, TestPoint:TestPoint_Pad_D1.0mm, symbol Connector:TestPoint
- removed U8: FE1.1s, Package_SO:SSOP-28_3.9x9.9mm_P0.635mm, symbol Interface_USB:FE1.1s
- added C37, C42: 1u, Capacitor_SMD:C_0805_2012Metric, symbol Device:C_Small
- added R16: 100k, Resistor_SMD:R_0603_1608Metric, symbol Device:R_Small
- added R45: 10k, Resistor_SMD:R_0603_1608Metric, symbol Device:R_Small
- added U3: LP5907MFX-3.3, Package_TO_SOT_SMD:SOT-23-5, symbol Regulator_Linear:LP5907MFX-3.3
- added U8: FE1.1s-BQFN24B, Package_DFN_QFN:QFN-24-1EP_4x4mm_P0.5mm_EP2.6x2.6mm_ThermalVias, symbol ZOUDIOsymbols:FE1.1s-BQFN24B
- F1: footprint (none) -> Fuse:Fuse_1206_3216Metric
- Y2: renamed from Y1; symbol Device:Crystal_GND23_Small -> Device:Crystal_GND24_Small
- renumbered C55 to C36, D7 to D1, FB5 to FB1, FB1 to FB2, FB2 to FB3, FB3 to FB4, FB4 to FB5, J4 to J8, R38 to R18, R39 to R19, R1 to R20, R6 to R21, TP4 to TP3
Connections:
- net 3V3: now also C36.2, R18.1, C42.1, R16.1, R45.1, U3.5 (OUT), U8.20 (VD33F)
- net DRV: now also R21.1, U8.21 (DRV); no longer D1.2 (A)
- net GND: now also D1.1 (K), Y2.4, C37.2, C42.2, U3.2 (GND), U8.25 (EP); no longer R21.2, Y2.3
- net I2C_SCL: now also TP2.1, U8.22 (LED1); no longer TP1.1
- net I2C_SDA: now also TP1.1, U8.2 (TESTJ); no longer TP2.1
- net LED2: now also U8.23 (LED2)
- net at R18.2: now also U8.16 (XRSTJ)
- net at R19.2: now also U8.18 (BUSJ)
- net at Y2.1: now also U8.3 (XOUT)
- net at FB3.2: now also U8.11 (DM1)
- net at FB2.2: now also U8.12 (DP1)
- net at FB5.2: now also U8.9 (DM2)
- net at FB4.2: now also U8.10 (DP2)
- net at J8.2 (D-): now also U8.14 (DMU)
- net at J8.3 (D+): now also U8.15 (DPU)
- net at R20.2: now also U8.13 (REXT)
- removed net +5V: C36.2, F1.1, R18.1
- net DM1 renamed D1-
- net DM2 renamed D2-
- net DP1 renamed D1+
- net DP2 renamed D2+
- new net: U8.4 (XIN), Y2.3
- new net: D1.2 (A), R21.2
- new net: R45.2, U8.1 (OVCJ)
- new net: R16.2, U8.17 (VBUSM)
- new net 5V_usb: C37.1, F1.1, U3.1 (IN), U3.3 (EN)
- no-connect marks 6 -> 7
Other:
- note added: "3.3V LDO"
- moved on the sheet: C36, D1, F1, FB1, FB2, FB3, FB4, FB5, J8, R18, R19, R20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
