File: Hardware/User controls.sch (KiCad schematic (older format))
At the start: 9 parts

Commit message: Pre refdes fix
Parts:
- removed C?: 100n, ZOUDIOfootprints:C0603, symbol Device:C_Small
- removed R?: 10K, ZOUDIOfootprints:R0603, symbol Device:R_Small
- J5, J6: renamed from J?; footprint ZOUDIOfootprints:JSTPH_2P -> Connector_JST:JST_PH_B2B-PH-K_1x02_P2.00mm_Vertical
- J7: renamed from J?; footprint ZOUDIOfootprints:JSTPH_10P -> Connector_JST:JST_PH_B10B-PH-K_1x10_P2.00mm_Vertical
- R2, R3, R5: renamed from R?; value 100K -> 100k; footprint ZOUDIOfootprints:R0603 -> Resistor_SMD:R_0603_1608Metric
- R4: renamed from R?; footprint ZOUDIOfootprints:R0603 -> Resistor_SMD:R_0603_1608Metric
Connections:
- net +3V3: now also J7.7 (Pin_7); no longer J7.4 (Pin_4)
- net AUX_GND: now also J7.9 (Pin_9); no longer J7.2 (Pin_2)
- net AUX_L: now also J7.10 (Pin_10); no longer J7.1 (Pin_1)
- net AUX_R: now also J7.8 (Pin_8); no longer J7.3 (Pin_3)
- net GND: now also J7.4 (Pin_4); no longer J7.7 (Pin_7)
- net LED_RED: now also J7.2 (Pin_2); no longer J7.9 (Pin_9)
- net ROT_A: now also J7.3 (Pin_3); no longer J7.8 (Pin_8)
- net ROT_B: now also J7.5 (Pin_5); no longer J7.6 (Pin_6)
- net ROT_SW: now also J7.6 (Pin_6), R5.2
- net at R4.1: now also J7.1 (Pin_1); no longer J7.10 (Pin_10)
Other:
- moved on the sheet: J5, J6, J7, R2, R3, R4, R5

Commit message: V0.1 check
Parts:
- R24: renamed from R4; value 100R -> 1k
- renumbered J7 to J2, R2 to R22, R3 to R23, R5 to R25
Connections:
- net AUX_L: now also J2.8 (Pin_8); no longer J2.10 (Pin_10)
- net AUX_R: now also J2.10 (Pin_10); no longer J2.8 (Pin_8)
Other:
- moved on the sheet: R25
Changed lines of the file:
@@
 $Descr A4 11693 8268
 encoding utf-8
-Sheet 6 9
+Sheet 8 9
 Title "4x38W amp with DSP and BT"
 Date "2021-06-08"
-Rev "V0.1"
+Rev "0.1"
 Comp "ZOUDIO"
 Comment1 ""
@@
 P 5300 3800
 AR Path="/60BE65E1" Ref="R?"  Part="1"
-AR Path="/60BE11E8/60BE65E1" Ref="R3"  Part="1"
-F 0 "R3" H 5350 3850 50  0000 L CNN
+AR Path="/60BE11E8/60BE65E1" Ref="R23"  Part="1"
+F 0 "R23" H 5350 3850 50  0000 L CNN
 F 1 "100k" H 5350 3750 50  0000 L CNN
 F 2 "Resistor_SMD:R_0603_1608Metric" H 5300 3800 50  0001 C CNN
@@
 P 5300 3550
 AR Path="/60BE65E7" Ref="#PWR?"  Part="1"
-AR Path="/60BE11E8/60BE65E7" Ref="#PWR0150"  Part="1"
-F 0 "#PWR0150" H 5300 3400 50  0001 C CNN
+AR Path="/60BE11E8/60BE65E7" Ref="#PWR0176"  Part="1"
+F 0 "#PWR0176" H 5300 3400 50  0001 C CNN
 F 1 "+3V3" V 5300 3750 50  0000 C CNN
 F 2 "" H 5300 3550 50  0001 C CNN
@@
 P 5300 3950
 AR Path="/60BE65FA" Ref="#PWR?"  Part="1"
-AR Path="/60BE11E8/60BE65FA" Ref="#PWR0151"  Part="1"
-F 0 "#PWR0151" H 5300 3700 50  0001 C CNN
+AR Path="/60BE11E8/60BE65FA" Ref="#PWR0177"  Part="1"
+F 0 "#PWR0177" H 5300 3700 50  0001 C CNN
 F 1 "GND" H 5305 3777 50  0001 C CNN
 F 2 "" H 5300 3950 50  0001 C CNN
@@
 P 5300 2850
 AR Path="/60BE6603" Ref="#PWR?"  Part="1"
-AR Path="/60BE11E8/60BE6603" Ref="#PWR0194"  Part="1"
-F 0 "#PWR0194" H 5300 2700 50  0001 C CNN
+AR Path="/60BE11E8/60BE6603" Ref="#PWR0178"  Part="1"
+F 0 "#PWR0178" H 5300 2700 50  0001 C CNN
 F 1 "+3V3" V 5300 3050 50  0000 C CNN
 F 2 "" H 5300 2850 50  0001 C CNN
@@
 P 5300 3250
 AR Path="/60BE6609" Ref="#PWR?"  Part="1"
-AR Path="/60BE11E8/60BE6609" Ref="#PWR0195"  Part="1"
-F 0 "#PWR0195" H 5300 3000 50  0001 C CNN
+AR Path="/60BE11E8/60BE6609" Ref="#PWR0179"  Part="1"
+F 0 "#PWR0179" H 5300 3000 50  0001 C CNN
 F 1 "GND" H 5305 3077 50  0001 C CNN
 F 2 "" H 5300 3250 50  0001 C CNN
@@
 P 5300 3100
 AR Path="/60BE660F" Ref="R?"  Part="1"
-AR Path="/60BE11E8/60BE660F" Ref="R2"  Part="1"
-F 0 "R2" H 5350 3150 50  0000 L CNN
+AR Path="/60BE11E8/60BE660F" Ref="R22"  Part="1"
+F 0 "R22" H 5350 3150 50  0000 L CNN
 F 1 "100k" H 5350 3050 50  0000 L CNN
 F 2 "Resistor_SMD:R_0603_1608Metric" H 5300 3100 50  0001 C CNN
@@
 Text HLabel 5550 4900 2    50   Output ~ 0
 ROT_B
-Text HLabel 6250 5000 2    50   Output ~ 0
+Text HLabel 6200 5000 2    50   Output ~ 0
 ROT_SW
-Text HLabel 5550 5200 2    50   Output ~ 0
+Text HLabel 5550 5400 2    50   Output ~ 0
 AUX_R
 Text HLabel 5550 5300 2    50   Output ~ 0
 AUX_GND
-Text HLabel 5550 5400 2    50   Output ~ 0
+Text HLabel 5550 5200 2    50   Output ~ 0
 AUX_L
 Wire Wire Line
@@
 	5250 5000 6150 5000
 Wire Wire Line
-	6150 5000 6250 5000
-Connection ~ 6150 5000
-Wire Wire Line
-	6150 4950 6150 5000
-Wire Wire Line
-	6150 4700 6150 4750
+	6150 5300 6150 5250
 Wire Wire Line
 	5250 4700 5550 4700
@@
 L power:GND #PWR?
 U 1 1 60BE2AED
-P 6150 4700
+P 6150 5300
 AR Path="/60BE2AED" Ref="#PWR?"  Part="1"
-AR Path="/60BE11E8/60BE2AED" Ref="#PWR0135"  Part="1"
-F 0 "#PWR0135" H 6150 4450 50  0001 C CNN
-F 1 "GND" H 6155 4527 50  0001 C CNN
-F 2 "" H 6150 4700 50  0001 C CNN
-F 3 "" H 6150 4700 50  0001 C CNN
-	1    6150 4700
+AR Path="/60BE11E8/60BE2AED" Ref="#PWR0180"  Part="1"
+F 0 "#PWR0180" H 6150 5050 50  0001 C CNN
+F 1 "GND" H 6155 5127 50  0001 C CNN
+F 2 "" H 6150 5300 50  0001 C CNN
+F 3 "" H 6150 5300 50  0001 C CNN
+	1    6150 5300
+	1    0    0    -1
+$EndComp
+$Comp
+L Device:R_Small R?
+U 1 1 60BE2AE7
+P 6150 5150
+AR Path="/60BE2AE7" Ref="R?"  Part="1"
+AR Path="/60BE11E8/60BE2AE7" Ref="R25"  Part="1"
+F 0 "R25" H 5950 5100 50  0000 L CNN
+F 1 "100k" H 5900 5200 50  0000 L CNN
+F 2 "Resistor_SMD:R_0603_1608Metric" H 6150 5150 50  0001 C CNN
+F 3 "~" H 6150 5150 50  0001 C CNN
+	1    6150 5150
 	-1   0    0    1
-$EndComp
-$Comp
-L Device:R_Small R?
-U 1 1 60BE2AE7
-P 6150 4850
-AR Path="/60BE2AE7" Ref="R?"  Part="1"
-AR Path="/60BE11E8/60BE2AE7" Ref="R5"  Part="1"
-F 0 "R5" H 6200 4800 50  0000 L CNN
-F 1 "100k" H 6200 4900 50  0000 L CNN
-F 2 "Resistor_SMD:R_0603_1608Metric" H 6150 4850 50  0001 C CNN
-F 3 "~" H 6150 4850 50  0001 C CNN
-	1    6150 4850
-	1    0    0    -1
 $EndComp
 $Comp
@@
 P 5300 5100
 AR Path="/60BE2AE1" Ref="#PWR?"  Part="1"
-AR Path="/60BE11E8/60BE2AE1" Ref="#PWR0134"  Part="1"
-F 0 "#PWR0134" H 5300 4950 50  0001 C CNN
+AR Path="/60BE11E8/60BE2AE1" Ref="#PWR0181"  Part="1"
+F 0 "#PWR0181" H 5300 4950 50  0001 C CNN
 F 1 "+3V3" V 5300 5300 50  0000 C CNN
 F 2 "" H 5300 5100 50  0001 C CNN
@@
 P 5300 4800
 AR Path="/60BE2ADA" Ref="#PWR?"  Part="1"
-AR Path="/60BE11E8/60BE2ADA" Ref="#PWR0133"  Part="1"
-F 0 "#PWR0133" H 5300 4550 50  0001 C CNN
+AR Path="/60BE11E8/60BE2ADA" Ref="#PWR0182"  Part="1"
+F 0 "#PWR0182" H 5300 4550 50  0001 C CNN
 F 1 "GND" H 5305 4627 50  0001 C CNN
 F 2 "" H 5300 4800 50  0001 C CNN
@@
 P 5400 4500
 AR Path="/60BE2AD2" Ref="R?"  Part="1"
-AR Path="/60BE11E8/60BE2AD2" Ref="R4"  Part="1"
-F 0 "R4" V 5500 4450 50  0000 L CNN
-F 1 "100R" V 5600 4400 50  0000 L CNN
+AR Path="/60BE11E8/60BE2AD2" Ref="R24"  Part="1"
+F 0 "R24" V 5600 4450 50  0000 L CNN
+F 1 "1k" V 5500 4450 50  0000 L CNN
 F 2 "Resistor_SMD:R_0603_1608Metric" H 5400 4500 50  0001 C CNN
 F 3 "~" H 5400 4500 50  0001 C CNN
@@
 P 5050 4900
 AR Path="/60BE2B19" Ref="J?"  Part="1"
-AR Path="/60BE11E8/60BE2B19" Ref="J7"  Part="1"
-F 0 "J7" H 5200 4950 50  0000 C CNN
+AR Path="/60BE11E8/60BE2B19" Ref="J2"  Part="1"
+F 0 "J2" H 5200 4950 50  0000 C CNN
 F 1 "JST-PH 01x10" H 5400 4850 50  0000 C CNN
 F 2 "Connector_JST:JST_PH_B10B-PH-K_1x10_P2.00mm_Vertical" H 5050 4900 50  0001 C CNN
@@
 	-1   0    0    -1
 $EndComp
+Wire Wire Line
+	6150 5050 6150 5000
+Wire Wire Line
+	6200 5000 6150 5000
+Connection ~ 6150 5000
 $EndSCHEMATC
