File: Hardware/AIO438.sch (KiCad schematic (older format))
At the start: 0 parts

Commit message: Pre refdes fix
Other:
- note added: "Fiducials\nMounting\nSilkscreen logo"
- note removed: "Silkscreen logo\nMounting\nFiducials"

Commit message: V0.1 check
Other:
- note added: "Todo:\nCheck pinout JSTs against AIO4CH"

Commit message: Version 0.1
Changed lines of the file:
@@
 F3 "AUX_GND" O R 4850 5200 50
 F4 "AUX_R" O R 4850 5300 50
-F5 "ROT_SW" O R 4850 4450 50
+F5 "ROT_SW" O R 4850 4650 50
 F6 "ROT_B" O R 4850 4550 50
-F7 "ROT_A" O R 4850 4650 50
+F7 "ROT_A" O R 4850 4450 50
 F8 "LED_RED" I R 4850 4350 50
 F9 "LED_GREEN" I R 4850 4250 50
@@
 F7 "I2C_SDA" B R 6400 3050 50
 F8 "PD2" I R 6400 4100 50
-F9 "PD3" I R 6400 3300 50
-F10 "PC1" O R 6400 3500 50
-F11 "PC0" I L 5350 4850 50
-F12 "PD4" O R 6400 2750 50
-F13 "PE0" O R 6400 2650 50
-F14 "PD6" O L 5350 4350 50
-F15 "PD5" O L 5350 4250 50
-F16 "UART_TX" O L 5350 2650 50
-F17 "UART_RX" I L 5350 2750 50
-F18 "PB0" I L 5350 4550 50
-F19 "PB1" O R 6400 3900 50
-F20 "PB2" O R 6400 3800 50
-F21 "PB3" I L 5350 4050 50
-F22 "PB4" I L 5350 4450 50
-F23 "DTR" I L 5350 2850 50
-F24 "PD7" I L 5350 4650 50
-F25 "PE2" I R 6400 3700 50
-F26 "PB5" I L 5350 3850 50
+F9 "PC1" O R 6400 3500 50
+F10 "PC0" I L 5350 4850 50
+F11 "PD4" O R 6400 2750 50
+F12 "PE0" O R 6400 2650 50
+F13 "PD6" O L 5350 4350 50
+F14 "PD5" O L 5350 4250 50
+F15 "UART_TX" O L 5350 2650 50
+F16 "UART_RX" I L 5350 2750 50
+F17 "PB0" I L 5350 4550 50
+F18 "PB1" O R 6400 3900 50
+F19 "PB2" O R 6400 3800 50
+F20 "PB3" I L 5350 4050 50
+F21 "PB4" I L 5350 4650 50
+F22 "DTR" I L 5350 2850 50
+F23 "PD7" I L 5350 4450 50
+F24 "PB5" I L 5350 3850 50
+F25 "PE2" O R 6400 3700 50
+F26 "PD3" O R 6400 3300 50
 $EndSheet
 $EndSCHEMATC
