File: Hardware/Microcontroller.sch (KiCad schematic (older format))
At the start: 14 parts, among them J11 PinHeader 02x03, J12 PinHeader 01x05, Q3 N-channel, U5 ATMEGA328PB, U6 M24256 EEPROM

Commit message: Pre refdes fix
Parts:
- removed U5: ATMEGA328PB, ZOUDIOfootprints:TQFP-32_7x7mm_Pitch0.8mm, symbol ZOUDIOsymbols:ATMEGA328PB
- added C42, C52: 18p, Capacitor_SMD:C_0603_1608Metric, symbol Device:C_Small
- added U12: ATmega328PB-AU, Package_QFP:TQFP-32_7x7mm_P0.8mm, symbol MCU_Microchip_ATmega:ATmega328PB-AU
- added Y2: 8MHz, Crystal:Crystal_SMD_Abracon_ABM3C-4Pin_5.0x3.2mm, symbol Device:Crystal_GND23_Small
- C49, C50: footprint ZOUDIOfootprints:C0603 -> Capacitor_SMD:C_0603_1608Metric
- J11: Function ISCP -> ICSP
- Q3: footprint ZOUDIOfootprints:SOT-23 -> Package_TO_SOT_SMD:SOT-23
- R25, R26, R27, R28, R29, R30, R31: footprint ZOUDIOfootprints:R0603 -> Resistor_SMD:R_0603_1608Metric
- U6: footprint ZOUDIOfootprints:TSSOP-8_4.4x3mm_P0.65mm -> Package_SO:TSSOP-8_4.4x3mm_P0.65mm
Connections:
- net +3V3: now also U12.18 (AVCC), U12.4 (VCC)
- net GND: now also C42.2, C52.2, U12.21 (GND), U12.5 (GND), Y2.2, Y2.3
- net I2C_SCL: now also U12.28 (PC5)
- net I2C_SDA: now also U12.27 (PC4)
- net PB0: now also U12.12 (PB0)
- net PB1: now also U12.13 (PB1)
- net PB2: now also U12.14 (PB2)
- net PC0: now also U12.23 (PC0)
- net PC1: now also U12.24 (PC1)
- net PC2: now also U12.25 (PC2)
- net PC3: now also U12.26 (PC3)
- net PD2: now also U12.32 (PD2)
- net PD3: now also U12.1 (PD3)
- net PD4: now also U12.2 (PD4)
- net PD5: now also U12.9 (PD5)
- net PD6: now also U12.10 (PD6)
- net PD7: now also U12.11 (PD7)
- net PE0: now also U12.3 (PE0)
- net PE1: now also U12.6 (PE1)
- net PE2: now also U12.19 (PE2)
- net PE3: now also U12.22 (PE3)
- net RESET: now also U12.29 (~RESET~/PC6)
- net SPI_CLK0: now also U12.17 (PB5)
- net SPI_MISO0: now also U12.16 (PB4)
- net SPI_MOSI0: now also U12.15 (PB3)
- net UART_RX: now also U12.30 (PD0)
- net UART_TX: now also U12.31 (PD1)
- new net XTAL1: C42.1, U12.7 (XTAL1/PB6), Y2.4
- new net XTAL2: C52.1, U12.8 (XTAL2/PB7), Y2.1
Other:
- note added: "*Pin 21 is hidden"
- note added: "Crystal"

Commit message: V0.1 check
Parts:
- removed Q3: N-channel, Package_TO_SOT_SMD:SOT-23, symbol ZOUDIOsymbols:N-Channel_SOT23
- added Q2: N-channel, Package_TO_SOT_SMD:SOT-23, symbol Device:Q_NMOS_GSD
- J3: renamed from J11; footprint ZOUDIOfootprints:PinSocket_2x03_P2.54mm_Vertical -> Connector_PinHeader_2.54mm:PinHeader_2x03_P2.54mm_Vertical
- J7: renamed from J12; value PinHeader 01x05 -> PinHeader 01x06; footprint ZOUDIOfootprints:PinHeader_1x05_P2.54mm_Vertical -> Connector_JST:JST_PH_B6B-PH-K_1x06_P2.00mm_Vertical; symbol Connector_Generic:Conn_01x05 -> Connector_Generic:Conn_01x06
- Y1: renamed from Y2; symbol Device:Crystal_GND23_Small -> Device:Crystal_GND24_Small
- renumbered C49 to C17, C42 to C34, C52 to C35, C50 to C54, R26 to R11, R27 to R12, R28 to R13, R30 to R14, R31 to R15, R25 to R2, R29 to R4, U12 to U6, U6 to U7
Connections:
- net +3V3: now also J3.2 (Pin_2), J7.4 (Pin_4); no longer J3.1 (Pin_1), J7.3 (Pin_3)
- net GND: now also J3.6 (Pin_6), Y1.4, Q2.2 (S); no longer J3.5 (Pin_5), Y1.3
- net I2C_SCL: now also J7.6 (Pin_6); no longer J7.5 (Pin_5)
- net I2C_SDA: now also J7.5 (Pin_5); no longer J7.4 (Pin_4)
- net PE1: now also Q2.1 (G)
- net RESET: now also J3.5 (Pin_5); no longer J3.6 (Pin_6)
- net SPI_CLK0: now also J3.3 (Pin_3); no longer J3.4 (Pin_4)
- net SPI_MISO0: now also J3.1 (Pin_1); no longer J3.2 (Pin_2)
- net SPI_MOSI0: now also J3.4 (Pin_4); no longer J3.3 (Pin_3)
- net XTAL1: now also Y1.3; no longer Y1.4
- net at J7.2 (Pin_2): now also Q2.3 (D)
- new net +5V: J7.3 (Pin_3)
Other:
- moved on the sheet: C17, C54, R11, R12, R13, R14, R15, R2, R4, U6

Commit message: Version 0.1
Changed lines of the file:
@@
 Text HLabel 4150 4600 2    50   Input ~ 0
 PD2
-Text HLabel 4150 4700 2    50   Input ~ 0
+Text HLabel 4150 4700 2    50   Output ~ 0
 PD3
 Text HLabel 4150 3700 2    50   Output ~ 0
@@
 Text HLabel 4150 5100 2    50   Input ~ 0
 PD7
-Text HLabel 2950 4600 0    50   Input ~ 0
+Text HLabel 2950 4600 0    50   Output ~ 0
 PE2
 Text Notes 4550 2700 0    50   ~ 0
