File: Mainboard/Amplifier.sch (KiCad schematic (older format))
At the start: 25 parts, among them U1 TAS5825M

Commit message: Result after weekend of lay-out
Pretty far, just neats to be cleaned up for production.
Does not pass DRC yet.
Changed lines of the file:
@@
 $Descr A4 11693 8268
 encoding utf-8
-Sheet 6 11
+Sheet 5 11
 Title "4x38W amp with DSP and BT"
 Date "2021-11-19"
@@
 AR Path="/60AAD6DF/61D69C28/61D73CD8" Ref="C39"  Part="1"
 AR Path="/60AAD6DF/61DB323F/61D73CD8" Ref="C3"  Part="1"
-F 0 "C3" H 4850 2450 50  0000 C CNN
+F 0 "C39" H 4850 2450 50  0000 C CNN
 F 1 "100n" H 4850 2550 50  0000 C CNN
 F 2 "Capacitor_SMD:C_0603_1608Metric" H 5000 2450 50  0001 C CNN
@@
 AR Path="/60AAD6DF/61D69C28/61D73D33" Ref="C59"  Part="1"
 AR Path="/60AAD6DF/61DB323F/61D73D33" Ref="C58"  Part="1"
-F 0 "C58" H 3800 2450 50  0000 C CNN
+F 0 "C59" H 3800 2450 50  0000 C CNN
 F 1 "22u" H 3800 2550 50  0000 C CNN
 F 2 "Capacitor_SMD:C_0805_2012Metric" H 3950 2450 50  0001 C CNN
@@
 AR Path="/60AAD6DF/61D69C28/61D73D2D" Ref="C56"  Part="1"
 AR Path="/60AAD6DF/61DB323F/61D73D2D" Ref="C55"  Part="1"
-F 0 "C55" H 3450 2450 50  0000 C CNN
+F 0 "C56" H 3450 2450 50  0000 C CNN
 F 1 "22u" H 3450 2550 50  0000 C CNN
 F 2 "Capacitor_SMD:C_0805_2012Metric" H 3600 2450 50  0001 C CNN
@@
 AR Path="/60AAD6DF/61D69C28/61D73CF4" Ref="C19"  Part="1"
 AR Path="/60AAD6DF/61DB323F/61D73CF4" Ref="C57"  Part="1"
-F 0 "C57" H 3450 3750 50  0000 C CNN
+F 0 "C19" H 3450 3750 50  0000 C CNN
 F 1 "4.7u" H 3450 3850 50  0000 C CNN
 F 2 "Capacitor_SMD:C_0805_2012Metric" H 3600 3750 50  0001 C CNN
@@
 AR Path="/60AAD6DF/61D69C28/61D73CE8" Ref="C53"  Part="1"
 AR Path="/60AAD6DF/61DB323F/61D73CE8" Ref="C52"  Part="1"
-F 0 "C52" H 5550 2450 50  0000 C CNN
+F 0 "C53" H 5550 2450 50  0000 C CNN
 F 1 "22u" H 5550 2550 50  0000 C CNN
 F 2 "Capacitor_SMD:C_0805_2012Metric" H 5700 2450 50  0001 C CNN
@@
 AR Path="/60AAD6DF/61D69C28/61D73CE2" Ref="C41"  Part="1"
 AR Path="/60AAD6DF/61DB323F/61D73CE2" Ref="C40"  Part="1"
-F 0 "C40" H 5200 2450 50  0000 C CNN
+F 0 "C41" H 5200 2450 50  0000 C CNN
 F 1 "22u" H 5200 2550 50  0000 C CNN
 F 2 "Capacitor_SMD:C_0805_2012Metric" H 5350 2450 50  0001 C CNN
@@
 AR Path="/60AAD6DF/61D69C28/61D73CD2" Ref="C18"  Part="1"
 AR Path="/60AAD6DF/61DB323F/61D73CD2" Ref="C2"  Part="1"
-F 0 "C2" H 4150 2450 50  0000 C CNN
+F 0 "C18" H 4150 2450 50  0000 C CNN
 F 1 "100n" H 4150 2550 50  0000 C CNN
 F 2 "Capacitor_SMD:C_0603_1608Metric" H 4300 2450 50  0001 C CNN
@@
 AR Path="/60AAD6DF/61D69C28/61D73CCC" Ref="C38"  Part="1"
 AR Path="/60AAD6DF/61DB323F/61D73CCC" Ref="C4"  Part="1"
-F 0 "C4" H 3800 3750 50  0000 C CNN
+F 0 "C38" H 3800 3750 50  0000 C CNN
 F 1 "100n" H 3800 3850 50  0000 C CNN
 F 2 "Capacitor_SMD:C_0603_1608Metric" H 3950 3750 50  0001 C CNN
@@
 AR Path="/60AAD6DF/61D69C28/625155DD" Ref="TP4"  Part="1"
 AR Path="/60AAD6DF/61DB323F/625155DD" Ref="TP5"  Part="1"
-F 0 "TP5" V 4950 4950 50  0000 C CNN
+F 0 "TP4" V 4950 4950 50  0000 C CNN
 F 1 "TestPoint" V 4850 5050 50  0000 C CNN
 F 2 "TestPoint:TestPoint_Pad_D1.0mm" H 5100 4700 50  0001 C CNN
@@
 AR Path="/60AAD6DF/61DB323F/61A2F14F" Ref="U1"  Part="1"
 AR Path="/60AAD6DF/61D69C28/61A2F14F" Ref="U2"  Part="1"
-F 0 "U1" H 5200 5400 50  0000 C CNN
+F 0 "U2" H 5200 5400 50  0000 C CNN
 F 1 "TAS5825M" H 6050 5400 50  0000 C CNN
 F 2 "ZOUDIO-footprints:TAS5825M" H 5700 4300 50  0001 C CNN
@@
 AR Path="/60AAD6DF/61D69C28/61D73CA4" Ref="C16"  Part="1"
 AR Path="/60AAD6DF/61DB323F/61D73CA4" Ref="C32"  Part="1"
-F 0 "C32" H 7550 4400 50  0000 C CNN
+F 0 "C16" H 7550 4400 50  0000 C CNN
 F 1 "680n" H 7550 4500 50  0000 C CNN
 F 2 "Capacitor_SMD:C_0805_2012Metric" H 7700 4400 50  0001 C CNN
@@
 AR Path="/60AAD6DF/61D69C28/61D73BEA" Ref="C26"  Part="1"
 AR Path="/60AAD6DF/61DB323F/61D73BEA" Ref="C8"  Part="1"
-F 0 "C8" V 6450 3250 50  0000 C CNN
+F 0 "C26" V 6450 3250 50  0000 C CNN
 F 1 "470n" V 6550 3250 50  0000 C CNN
 F 2 "Capacitor_SMD:C_0603_1608Metric" H 6500 3100 50  0001 C CNN
@@
 AR Path="/60AAD6DF/61D69C28/61D73BF6" Ref="C27"  Part="1"
 AR Path="/60AAD6DF/61DB323F/61D73BF6" Ref="C9"  Part="1"
-F 0 "C9" V 6450 3750 50  0000 C CNN
+F 0 "C27" V 6450 3750 50  0000 C CNN
 F 1 "470n" V 6550 3750 50  0000 C CNN
 F 2 "Capacitor_SMD:C_0603_1608Metric" H 6500 3600 50  0001 C CNN
@@
 AR Path="/60AAD6DF/61D69C28/61D73BFC" Ref="C28"  Part="1"
 AR Path="/60AAD6DF/61DB323F/61D73BFC" Ref="C10"  Part="1"
-F 0 "C10" V 6450 4050 50  0000 C CNN
+F 0 "C28" V 6450 4050 50  0000 C CNN
 F 1 "470n" V 6550 4050 50  0000 C CNN
 F 2 "Capacitor_SMD:C_0603_1608Metric" H 6500 3900 50  0001 C CNN
@@
 AR Path="/60AAD6DF/61D69C28/61D73C02" Ref="C29"  Part="1"
 AR Path="/60AAD6DF/61DB323F/61D73C02" Ref="C11"  Part="1"
-F 0 "C11" V 6450 4550 50  0000 C CNN
+F 0 "C29" V 6450 4550 50  0000 C CNN
 F 1 "470n" V 6550 4550 50  0000 C CNN
 F 2 "Capacitor_SMD:C_0603_1608Metric" H 6500 4400 50  0001 C CNN
@@
 AR Path="/60AAD6DF/61D69C28/61D73C56" Ref="C30"  Part="1"
 AR Path="/60AAD6DF/61DB323F/61D73C56" Ref="C12"  Part="1"
-F 0 "C12" H 7150 3600 50  0000 C CNN
+F 0 "C30" H 7150 3600 50  0000 C CNN
 F 1 "680n" H 7150 3700 50  0000 C CNN
 F 2 "Capacitor_SMD:C_0805_2012Metric" H 7300 3600 50  0001 C CNN
@@
 AR Path="/60AAD6DF/61D69C28/61D73C5C" Ref="C33"  Part="1"
 AR Path="/60AAD6DF/61DB323F/61D73C5C" Ref="C14"  Part="1"
-F 0 "C14" H 7550 3600 50  0000 C CNN
+F 0 "C33" H 7550 3600 50  0000 C CNN
 F 1 "680n" H 7550 3700 50  0000 C CNN
 F 2 "Capacitor_SMD:C_0805_2012Metric" H 7700 3600 50  0001 C CNN
@@
 AR Path="/60AAD6DF/61D69C28/61D73C81" Ref="L8"  Part="1"
 AR Path="/60AAD6DF/61DB323F/61D73C81" Ref="L4"  Part="1"
-F 0 "L4" V 7250 4050 50  0000 C CNN
+F 0 "L8" V 7250 4050 50  0000 C CNN
 F 1 "10u" V 7150 4050 50  0000 C CNN
 F 2 "ZOUDIO-footprints:Murata_1274AS-H-100M" H 7050 4050 50  0001 C CNN
@@
 AR Path="/60AAD6DF/61D69C28/61D73C87" Ref="L9"  Part="1"
 AR Path="/60AAD6DF/61DB323F/61D73C87" Ref="L5"  Part="1"
-F 0 "L5" V 7000 4250 50  0000 C CNN
+F 0 "L9" V 7000 4250 50  0000 C CNN
 F 1 "10u" V 6900 4250 50  0000 C CNN
 F 2 "ZOUDIO-footprints:Murata_1274AS-H-100M" H 7050 4250 50  0001 C CNN
@@
 AR Path="/60AAD6DF/61D69C28/61D73C8D" Ref="L7"  Part="1"
 AR Path="/60AAD6DF/61DB323F/61D73C8D" Ref="L3"  Part="1"
-F 0 "L3" V 7000 3450 50  0000 C CNN
+F 0 "L7" V 7000 3450 50  0000 C CNN
 F 1 "10u" V 6900 3450 50  0000 C CNN
 F 2 "ZOUDIO-footprints:Murata_1274AS-H-100M" H 7050 3450 50  0001 C CNN
@@
 AR Path="/60AAD6DF/61D69C28/61D73C93" Ref="L6"  Part="1"
 AR Path="/60AAD6DF/61DB323F/61D73C93" Ref="L2"  Part="1"
-F 0 "L2" V 7250 3250 50  0000 C CNN
+F 0 "L6" V 7250 3250 50  0000 C CNN
 F 1 "10u" V 7150 3250 50  0000 C CNN
 F 2 "ZOUDIO-footprints:Murata_1274AS-H-100M" H 7050 3250 50  0001 C CNN
@@
 AR Path="/60AAD6DF/61D69C28/61D73C9E" Ref="C31"  Part="1"
 AR Path="/60AAD6DF/61DB323F/61D73C9E" Ref="C15"  Part="1"
-F 0 "C15" H 7150 4400 50  0000 C CNN
+F 0 "C31" H 7150 4400 50  0000 C CNN
 F 1 "680n" H 7150 4500 50  0000 C CNN
 F 2 "Capacitor_SMD:C_0805_2012Metric" H 7300 4400 50  0001 C CNN
@@
 AR Path="/60AAD6DF/61D69C28/61D73C2D" Ref="C25"  Part="1"
 AR Path="/60AAD6DF/61DB323F/61D73C2D" Ref="C7"  Part="1"
-F 0 "C7" V 4850 3900 50  0000 C CNN
+F 0 "C25" V 4850 3900 50  0000 C CNN
 F 1 "1u" V 4950 3900 50  0000 C CNN
 F 2 "Capacitor_SMD:C_0805_2012Metric" H 4900 3800 50  0001 C CNN
@@
 AR Path="/60AAD6DF/61D69C28/61D73C33" Ref="C24"  Part="1"
 AR Path="/60AAD6DF/61DB323F/61D73C33" Ref="C6"  Part="1"
-F 0 "C6" V 4650 4000 50  0000 C CNN
+F 0 "C24" V 4650 4000 50  0000 C CNN
 F 1 "1u" V 4750 4000 50  0000 C CNN
 F 2 "Capacitor_SMD:C_0805_2012Metric" H 4700 3900 50  0001 C CNN
@@
 AR Path="/60AAD6DF/61D69C28/61D73C39" Ref="C20"  Part="1"
 AR Path="/60AAD6DF/61DB323F/61D73C39" Ref="C5"  Part="1"
-F 0 "C5" V 4450 4100 50  0000 C CNN
+F 0 "C20" V 4450 4100 50  0000 C CNN
 F 1 "1u" V 4550 4100 50  0000 C CNN
 F 2 "Capacitor_SMD:C_0805_2012Metric" H 4500 4000 50  0001 C CNN

Commit message: Mainboard: Version 1.0
Still need to clean up 3D models and BoM list,
but gerberexport-ready and ready to order.
Parts:
- removed TP4: TestPoint, TestPoint:TestPoint_Pad_D1.0mm, symbol Connector:TestPoint
Connections:
- no-connect marks 2 -> 3
Changed lines of the file:
@@
 $Descr A4 11693 8268
 encoding utf-8
-Sheet 5 11
+Sheet 6 11
 Title "4x38W amp with DSP and BT"
-Date "2021-11-19"
-Rev "0.2"
+Date "2021-12-01"
+Rev "1.0"
 Comp "ZOUDIO"
 Comment1 ""
@@
 AR Path="/60AAD6DF/61D69C28/61D73CD8" Ref="C39"  Part="1"
 AR Path="/60AAD6DF/61DB323F/61D73CD8" Ref="C3"  Part="1"
-F 0 "C39" H 4850 2450 50  0000 C CNN
+F 0 "C3" H 4850 2450 50  0000 C CNN
 F 1 "100n" H 4850 2550 50  0000 C CNN
 F 2 "Capacitor_SMD:C_0603_1608Metric" H 5000 2450 50  0001 C CNN
@@
 AR Path="/60AAD6DF/61D69C28/61D73D33" Ref="C59"  Part="1"
 AR Path="/60AAD6DF/61DB323F/61D73D33" Ref="C58"  Part="1"
-F 0 "C59" H 3800 2450 50  0000 C CNN
+F 0 "C58" H 3800 2450 50  0000 C CNN
 F 1 "22u" H 3800 2550 50  0000 C CNN
 F 2 "Capacitor_SMD:C_0805_2012Metric" H 3950 2450 50  0001 C CNN
@@
 AR Path="/60AAD6DF/61D69C28/61D73D2D" Ref="C56"  Part="1"
 AR Path="/60AAD6DF/61DB323F/61D73D2D" Ref="C55"  Part="1"
-F 0 "C56" H 3450 2450 50  0000 C CNN
+F 0 "C55" H 3450 2450 50  0000 C CNN
 F 1 "22u" H 3450 2550 50  0000 C CNN
 F 2 "Capacitor_SMD:C_0805_2012Metric" H 3600 2450 50  0001 C CNN
@@
 AR Path="/60AAD6DF/61D69C28/61D73CF4" Ref="C19"  Part="1"
 AR Path="/60AAD6DF/61DB323F/61D73CF4" Ref="C57"  Part="1"
-F 0 "C19" H 3450 3750 50  0000 C CNN
+F 0 "C57" H 3450 3750 50  0000 C CNN
 F 1 "4.7u" H 3450 3850 50  0000 C CNN
 F 2 "Capacitor_SMD:C_0805_2012Metric" H 3600 3750 50  0001 C CNN
@@
 AR Path="/60AAD6DF/61D69C28/61D73CE8" Ref="C53"  Part="1"
 AR Path="/60AAD6DF/61DB323F/61D73CE8" Ref="C52"  Part="1"
-F 0 "C53" H 5550 2450 50  0000 C CNN
+F 0 "C52" H 5550 2450 50  0000 C CNN
 F 1 "22u" H 5550 2550 50  0000 C CNN
 F 2 "Capacitor_SMD:C_0805_2012Metric" H 5700 2450 50  0001 C CNN
@@
 AR Path="/60AAD6DF/61D69C28/61D73CE2" Ref="C41"  Part="1"
 AR Path="/60AAD6DF/61DB323F/61D73CE2" Ref="C40"  Part="1"
-F 0 "C41" H 5200 2450 50  0000 C CNN
+F 0 "C40" H 5200 2450 50  0000 C CNN
 F 1 "22u" H 5200 2550 50  0000 C CNN
 F 2 "Capacitor_SMD:C_0805_2012Metric" H 5350 2450 50  0001 C CNN
@@
 AR Path="/60AAD6DF/61D69C28/61D73CD2" Ref="C18"  Part="1"
 AR Path="/60AAD6DF/61DB323F/61D73CD2" Ref="C2"  Part="1"
-F 0 "C18" H 4150 2450 50  0000 C CNN
+F 0 "C2" H 4150 2450 50  0000 C CNN
 F 1 "100n" H 4150 2550 50  0000 C CNN
 F 2 "Capacitor_SMD:C_0603_1608Metric" H 4300 2450 50  0001 C CNN
@@
 AR Path="/60AAD6DF/61D69C28/61D73CCC" Ref="C38"  Part="1"
 AR Path="/60AAD6DF/61DB323F/61D73CCC" Ref="C4"  Part="1"
-F 0 "C38" H 3800 3750 50  0000 C CNN
+F 0 "C4" H 3800 3750 50  0000 C CNN
 F 1 "100n" H 3800 3850 50  0000 C CNN
 F 2 "Capacitor_SMD:C_0603_1608Metric" H 3950 3750 50  0001 C CNN
@@
 $EndComp
 $Comp
-L Connector:TestPoint TP4
-U 1 1 625155DD
-P 4900 4700
-AR Path="/60AAD6DF/61D69C28/625155DD" Ref="TP4"  Part="1"
-AR Path="/60AAD6DF/61DB323F/625155DD" Ref="TP5"  Part="1"
-F 0 "TP4" V 4950 4950 50  0000 C CNN
-F 1 "TestPoint" V 4850 5050 50  0000 C CNN
-F 2 "TestPoint:TestPoint_Pad_D1.0mm" H 5100 4700 50  0001 C CNN
-F 3 "~" H 5100 4700 50  0001 C CNN
-	1    4900 4700
-	0    -1   -1   0
-$EndComp
-Wire Wire Line
-	4900 4700 5050 4700
-$Comp
 L ZOUDIO-symbols:TAS5825M U1
 U 1 1 61A2F14F
@@
 AR Path="/60AAD6DF/61DB323F/61A2F14F" Ref="U1"  Part="1"
 AR Path="/60AAD6DF/61D69C28/61A2F14F" Ref="U2"  Part="1"
-F 0 "U2" H 5200 5400 50  0000 C CNN
+F 0 "U1" H 5200 5400 50  0000 C CNN
 F 1 "TAS5825M" H 6050 5400 50  0000 C CNN
 F 2 "ZOUDIO-footprints:TAS5825M" H 5700 4300 50  0001 C CNN
@@
 AR Path="/60AAD6DF/61D69C28/61D73CA4" Ref="C16"  Part="1"
 AR Path="/60AAD6DF/61DB323F/61D73CA4" Ref="C32"  Part="1"
-F 0 "C16" H 7550 4400 50  0000 C CNN
+F 0 "C32" H 7550 4400 50  0000 C CNN
 F 1 "680n" H 7550 4500 50  0000 C CNN
 F 2 "Capacitor_SMD:C_0805_2012Metric" H 7700 4400 50  0001 C CNN
@@
 AR Path="/60AAD6DF/61D69C28/61D73BEA" Ref="C26"  Part="1"
 AR Path="/60AAD6DF/61DB323F/61D73BEA" Ref="C8"  Part="1"
-F 0 "C26" V 6450 3250 50  0000 C CNN
+F 0 "C8" V 6450 3250 50  0000 C CNN
 F 1 "470n" V 6550 3250 50  0000 C CNN
 F 2 "Capacitor_SMD:C_0603_1608Metric" H 6500 3100 50  0001 C CNN
@@
 AR Path="/60AAD6DF/61D69C28/61D73BF6" Ref="C27"  Part="1"
 AR Path="/60AAD6DF/61DB323F/61D73BF6" Ref="C9"  Part="1"
-F 0 "C27" V 6450 3750 50  0000 C CNN
+F 0 "C9" V 6450 3750 50  0000 C CNN
 F 1 "470n" V 6550 3750 50  0000 C CNN
 F 2 "Capacitor_SMD:C_0603_1608Metric" H 6500 3600 50  0001 C CNN
@@
 AR Path="/60AAD6DF/61D69C28/61D73BFC" Ref="C28"  Part="1"
 AR Path="/60AAD6DF/61DB323F/61D73BFC" Ref="C10"  Part="1"
-F 0 "C28" V 6450 4050 50  0000 C CNN
+F 0 "C10" V 6450 4050 50  0000 C CNN
 F 1 "470n" V 6550 4050 50  0000 C CNN
 F 2 "Capacitor_SMD:C_0603_1608Metric" H 6500 3900 50  0001 C CNN
@@
 AR Path="/60AAD6DF/61D69C28/61D73C02" Ref="C29"  Part="1"
 AR Path="/60AAD6DF/61DB323F/61D73C02" Ref="C11"  Part="1"
-F 0 "C29" V 6450 4550 50  0000 C CNN
+F 0 "C11" V 6450 4550 50  0000 C CNN
 F 1 "470n" V 6550 4550 50  0000 C CNN
 F 2 "Capacitor_SMD:C_0603_1608Metric" H 6500 4400 50  0001 C CNN
@@
 AR Path="/60AAD6DF/61D69C28/61D73C56" Ref="C30"  Part="1"
 AR Path="/60AAD6DF/61DB323F/61D73C56" Ref="C12"  Part="1"
-F 0 "C30" H 7150 3600 50  0000 C CNN
+F 0 "C12" H 7150 3600 50  0000 C CNN
 F 1 "680n" H 7150 3700 50  0000 C CNN
 F 2 "Capacitor_SMD:C_0805_2012Metric" H 7300 3600 50  0001 C CNN
@@
 AR Path="/60AAD6DF/61D69C28/61D73C5C" Ref="C33"  Part="1"
 AR Path="/60AAD6DF/61DB323F/61D73C5C" Ref="C14"  Part="1"
-F 0 "C33" H 7550 3600 50  0000 C CNN
+F 0 "C14" H 7550 3600 50  0000 C CNN
 F 1 "680n" H 7550 3700 50  0000 C CNN
 F 2 "Capacitor_SMD:C_0805_2012Metric" H 7700 3600 50  0001 C CNN
@@
 AR Path="/60AAD6DF/61D69C28/61D73C81" Ref="L8"  Part="1"
 AR Path="/60AAD6DF/61DB323F/61D73C81" Ref="L4"  Part="1"
-F 0 "L8" V 7250 4050 50  0000 C CNN
+F 0 "L4" V 7250 4050 50  0000 C CNN
 F 1 "10u" V 7150 4050 50  0000 C CNN
 F 2 "ZOUDIO-footprints:Murata_1274AS-H-100M" H 7050 4050 50  0001 C CNN
@@
 AR Path="/60AAD6DF/61D69C28/61D73C87" Ref="L9"  Part="1"
 AR Path="/60AAD6DF/61DB323F/61D73C87" Ref="L5"  Part="1"
-F 0 "L9" V 7000 4250 50  0000 C CNN
+F 0 "L5" V 7000 4250 50  0000 C CNN
 F 1 "10u" V 6900 4250 50  0000 C CNN
 F 2 "ZOUDIO-footprints:Murata_1274AS-H-100M" H 7050 4250 50  0001 C CNN
@@
 AR Path="/60AAD6DF/61D69C28/61D73C8D" Ref="L7"  Part="1"
 AR Path="/60AAD6DF/61DB323F/61D73C8D" Ref="L3"  Part="1"
-F 0 "L7" V 7000 3450 50  0000 C CNN
+F 0 "L3" V 7000 3450 50  0000 C CNN
 F 1 "10u" V 6900 3450 50  0000 C CNN
 F 2 "ZOUDIO-footprints:Murata_1274AS-H-100M" H 7050 3450 50  0001 C CNN
@@
 AR Path="/60AAD6DF/61D69C28/61D73C93" Ref="L6"  Part="1"
 AR Path="/60AAD6DF/61DB323F/61D73C93" Ref="L2"  Part="1"
-F 0 "L6" V 7250 3250 50  0000 C CNN
+F 0 "L2" V 7250 3250 50  0000 C CNN
 F 1 "10u" V 7150 3250 50  0000 C CNN
 F 2 "ZOUDIO-footprints:Murata_1274AS-H-100M" H 7050 3250 50  0001 C CNN
@@
 AR Path="/60AAD6DF/61D69C28/61D73C9E" Ref="C31"  Part="1"
 AR Path="/60AAD6DF/61DB323F/61D73C9E" Ref="C15"  Part="1"
-F 0 "C31" H 7150 4400 50  0000 C CNN
+F 0 "C15" H 7150 4400 50  0000 C CNN
 F 1 "680n" H 7150 4500 50  0000 C CNN
 F 2 "Capacitor_SMD:C_0805_2012Metric" H 7300 4400 50  0001 C CNN
@@
 AR Path="/60AAD6DF/61D69C28/61D73C2D" Ref="C25"  Part="1"
 AR Path="/60AAD6DF/61DB323F/61D73C2D" Ref="C7"  Part="1"
-F 0 "C25" V 4850 3900 50  0000 C CNN
+F 0 "C7" V 4850 3900 50  0000 C CNN
 F 1 "1u" V 4950 3900 50  0000 C CNN
 F 2 "Capacitor_SMD:C_0805_2012Metric" H 4900 3800 50  0001 C CNN
@@
 AR Path="/60AAD6DF/61D69C28/61D73C33" Ref="C24"  Part="1"
 AR Path="/60AAD6DF/61DB323F/61D73C33" Ref="C6"  Part="1"
-F 0 "C24" V 4650 4000 50  0000 C CNN
+F 0 "C6" V 4650 4000 50  0000 C CNN
 F 1 "1u" V 4750 4000 50  0000 C CNN
 F 2 "Capacitor_SMD:C_0805_2012Metric" H 4700 3900 50  0001 C CNN
@@
 AR Path="/60AAD6DF/61D69C28/61D73C39" Ref="C20"  Part="1"
 AR Path="/60AAD6DF/61DB323F/61D73C39" Ref="C5"  Part="1"
-F 0 "C20" V 4450 4100 50  0000 C CNN
+F 0 "C5" V 4450 4100 50  0000 C CNN
 F 1 "1u" V 4550 4100 50  0000 C CNN
 F 2 "Capacitor_SMD:C_0805_2012Metric" H 4500 4000 50  0001 C CNN
@@
 Wire Wire Line
 	5050 3900 4800 3900
+NoConn ~ 5050 4700
 $EndSCHEMATC
