File: Mainboard/Amplifiers.sch (KiCad schematic (older format))
At the start: 53 parts, among them J1 JST-PH 01x03, J4 5mm screwterminal 01x12, J9 JST-PH 01x04, U1 TAS5825M, U2 TAS5825M

Commit message: Modify library references
As described in the README of the newly added libraries submodule.
Schematic and PCB are synced.

Hardware folder is renamed to mainboard
Any other PCBs can be put in their own subfolder in the gitrepo

Commit also swaps source/drain of Q1 because it appeared wrong for some
reason after updating all symbol/footprints.
Parts:
- C1: footprint ZOUDIOfootprints:Cap_Rad_D10_P5_horizontal -> ZOUDIO-footprints:Cap_Rad_D10_P5_horizontal
- J4: footprint ZOUDIOfootprints:Multicomp_12P_5mm -> ZOUDIO-footprints:Multicomp_12P_5mm
- L2, L3, L4, L5, L6, L7, L8, L9: footprint ZOUDIOfootprints:Murata_1274AS-H-100M -> ZOUDIO-footprints:Murata_1274AS-H-100M
- U1, U2: footprint ZOUDIOfootprints:TAS5825M -> ZOUDIO-footprints:TAS5825M; symbol ZOUDIOsymbols:TAS5825M -> ZOUDIO-symbols:TAS5825M
Changed lines of the file:
@@
 $EndComp
 $Comp
-L ZOUDIOsymbols:TAS5825M U1
+L ZOUDIO-symbols:TAS5825M U1
 U 1 1 60AF269F
 P 3700 2700
 F 0 "U1" H 3200 3900 50  0000 C CNN
 F 1 "TAS5825M" H 4050 3900 50  0000 C CNN
-F 2 "ZOUDIOfootprints:TAS5825M" H 3700 2800 50  0001 C CNN
+F 2 "ZOUDIO-footprints:TAS5825M" H 3700 2800 50  0001 C CNN
 F 3 "" H 3700 2800 50  0001 C CNN
 	1    3700 2700
@@
 F 0 "L4" V 5300 2450 50  0000 C CNN
 F 1 "10u" V 5200 2450 50  0000 C CNN
-F 2 "ZOUDIOfootprints:Murata_1274AS-H-100M" H 5100 2450 50  0001 C CNN
+F 2 "ZOUDIO-footprints:Murata_1274AS-H-100M" H 5100 2450 50  0001 C CNN
 F 3 "~" H 5100 2450 50  0001 C CNN
 	1    5100 2450
@@
 F 0 "L5" V 5050 2650 50  0000 C CNN
 F 1 "10u" V 4950 2650 50  0000 C CNN
-F 2 "ZOUDIOfootprints:Murata_1274AS-H-100M" H 5100 2650 50  0001 C CNN
+F 2 "ZOUDIO-footprints:Murata_1274AS-H-100M" H 5100 2650 50  0001 C CNN
 F 3 "~" H 5100 2650 50  0001 C CNN
 	1    5100 2650
@@
 F 0 "L3" V 5050 1950 50  0000 C CNN
 F 1 "10u" V 4950 1950 50  0000 C CNN
-F 2 "ZOUDIOfootprints:Murata_1274AS-H-100M" H 5100 1950 50  0001 C CNN
+F 2 "ZOUDIO-footprints:Murata_1274AS-H-100M" H 5100 1950 50  0001 C CNN
 F 3 "~" H 5100 1950 50  0001 C CNN
 	1    5100 1950
@@
 F 0 "L2" V 5300 1750 50  0000 C CNN
 F 1 "10u" V 5200 1750 50  0000 C CNN
-F 2 "ZOUDIOfootprints:Murata_1274AS-H-100M" H 5100 1750 50  0001 C CNN
+F 2 "ZOUDIO-footprints:Murata_1274AS-H-100M" H 5100 1750 50  0001 C CNN
 F 3 "~" H 5100 1750 50  0001 C CNN
 	1    5100 1750
@@
 $EndComp
 $Comp
-L ZOUDIOsymbols:TAS5825M U2
+L ZOUDIO-symbols:TAS5825M U2
 U 1 1 60B2F840
 P 3700 6000
@@
 F 0 "U2" H 3200 7200 50  0000 C CNN
 F 1 "TAS5825M" H 4050 7200 50  0000 C CNN
-F 2 "ZOUDIOfootprints:TAS5825M" H 3700 6100 50  0001 C CNN
+F 2 "ZOUDIO-footprints:TAS5825M" H 3700 6100 50  0001 C CNN
 F 3 "" H 3700 6100 50  0001 C CNN
 	1    3700 6000
@@
 F 0 "L8" V 5300 5750 50  0000 C CNN
 F 1 "10u" V 5200 5750 50  0000 C CNN
-F 2 "ZOUDIOfootprints:Murata_1274AS-H-100M" H 5100 5750 50  0001 C CNN
+F 2 "ZOUDIO-footprints:Murata_1274AS-H-100M" H 5100 5750 50  0001 C CNN
 F 3 "~" H 5100 5750 50  0001 C CNN
 	1    5100 5750
@@
 F 0 "L9" V 5050 5950 50  0000 C CNN
 F 1 "10u" V 4950 5950 50  0000 C CNN
-F 2 "ZOUDIOfootprints:Murata_1274AS-H-100M" H 5100 5950 50  0001 C CNN
+F 2 "ZOUDIO-footprints:Murata_1274AS-H-100M" H 5100 5950 50  0001 C CNN
 F 3 "~" H 5100 5950 50  0001 C CNN
 	1    5100 5950
@@
 F 0 "L7" V 5050 5250 50  0000 C CNN
 F 1 "10u" V 4950 5250 50  0000 C CNN
-F 2 "ZOUDIOfootprints:Murata_1274AS-H-100M" H 5100 5250 50  0001 C CNN
+F 2 "ZOUDIO-footprints:Murata_1274AS-H-100M" H 5100 5250 50  0001 C CNN
 F 3 "~" H 5100 5250 50  0001 C CNN
 	1    5100 5250
@@
 F 0 "L6" V 5300 5050 50  0000 C CNN
 F 1 "10u" V 5200 5050 50  0000 C CNN
-F 2 "ZOUDIOfootprints:Murata_1274AS-H-100M" H 5100 5050 50  0001 C CNN
+F 2 "ZOUDIO-footprints:Murata_1274AS-H-100M" H 5100 5050 50  0001 C CNN
 F 3 "~" H 5100 5050 50  0001 C CNN
 	1    5100 5050
@@
 F 0 "C1" H 7350 1500 50  0000 L CNN
 F 1 "820u" H 7315 1405 50  0000 L CNN
-F 2 "ZOUDIOfootprints:Cap_Rad_D10_P5_horizontal" H 7238 1300 50  0001 C CNN
+F 2 "ZOUDIO-footprints:Cap_Rad_D10_P5_horizontal" H 7238 1300 50  0001 C CNN
 F 3 "~" H 7200 1450 50  0001 C CNN
 	1    7200 1450
@@
 F 0 "J4" H 8600 1650 50  0000 C CNN
 F 1 "5mm screwterminal 01x12" H 9050 1550 50  0000 C CNN
-F 2 "ZOUDIOfootprints:Multicomp_12P_5mm" H 8450 1650 50  0001 C CNN
+F 2 "ZOUDIO-footprints:Multicomp_12P_5mm" H 8450 1650 50  0001 C CNN
 F 3 "~" H 8450 1650 50  0001 C CNN
 F 4 "Amp out / power in" H 8950 1450 50  0000 C CNN "Function"

Commit message: Before testing CH340B and VCHG
Cleaned up amp lay-out a bit in the meanwhile
Parts:
- removed C10, C11, C26, C27, C28, C29, C8, C9: 470n, Capacitor_SMD:C_0603_1608Metric, symbol Device:C_Small
- removed C12, C14, C15, C30, C31, C32, C33, C43: 680n, Capacitor_SMD:C_0805_2012Metric, symbol Device:C_Small
- removed C18, C2, C3, C38, C39, C4: 100n, Capacitor_SMD:C_0603_1608Metric, symbol Device:C_Small
- removed C19, C20, C24, C25, C5, C6, C7: 1u, Capacitor_SMD:C_0805_2012Metric, symbol Device:C_Small
- removed C40, C41, C52, C53, C55, C56, C58, C59: 22u, Capacitor_SMD:C_0805_2012Metric, symbol Device:C_Small
- removed C57: 4.7u, Capacitor_SMD:C_0805_2012Metric, symbol Device:C_Small
- removed L2, L3, L4, L5, L6, L7, L8, L9: 10u, ZOUDIO-footprints:Murata_1274AS-H-100M, symbol Device:L
- removed U1, U2: TAS5825M, ZOUDIO-footprints:TAS5825M, symbol ZOUDIO-symbols:TAS5825M
- C1: symbol Device:C -> Device:CP
Connections:
- net labels removed: +3V3
- wire segments 215 -> 53
- no-connect marks 6 -> 0
Other:
- note added: "0x4C"
- note added: "0x4D"
- note removed: "Amplifier 1"
- note removed: "Amplifier 2"
- note removed: "I2C address = 0x4C"
- note removed: "I2C address = 0x4D"
- note removed: "I2S"
- note removed: "Power connectors"
- moved on the sheet: J1, J9

Commit message: Result after weekend of lay-out
Pretty far, just neats to be cleaned up for production.
Does not pass DRC yet.
Parts:
- removed J9: JST-PH 01x04, Connector_JST:JST_PH_B4B-PH-K_1x04_P2.00mm_Vertical, symbol Connector_Generic:Conn_01x04
Changed lines of the file:
@@
 Wire Wire Line
 	6250 4000 7200 4000
-Text GLabel 7100 2600 0    50   Output ~ 0
-Vin
-$Comp
-L Connector_Generic:Conn_01x04 J?
-U 1 1 60C17FDF
-P 7400 2400
-AR Path="/60C17FDF" Ref="J?"  Part="1"
-AR Path="/60B7AC16/60C17FDF" Ref="J?"  Part="1"
-AR Path="/60AAD6DF/60C17FDF" Ref="J9"  Part="1"
-F 0 "J9" H 7500 2450 50  0000 L CNN
-F 1 "JST-PH 01x04" H 7500 2350 50  0000 L CNN
-F 2 "Connector_JST:JST_PH_B4B-PH-K_1x04_P2.00mm_Vertical" H 7400 2400 50  0001 C CNN
-F 3 "~" H 7400 2400 50  0001 C CNN
-F 4 "Sure BCPBx" H 7750 2250 50  0000 C CNN "Function"
-	1    7400 2400
-	1    0    0    -1
-$EndComp
-$Comp
-L power:GND #PWR?
-U 1 1 60C17FD9
-P 7100 2300
-AR Path="/60C17FD9" Ref="#PWR?"  Part="1"
-AR Path="/60B7AC16/60C17FD9" Ref="#PWR?"  Part="1"
-AR Path="/60AAD6DF/60C17FD9" Ref="#PWR0119"  Part="1"
-F 0 "#PWR0119" H 7100 2050 50  0001 C CNN
-F 1 "GND" H 7105 2127 50  0001 C CNN
-F 2 "" H 7100 2300 50  0001 C CNN
-F 3 "" H 7100 2300 50  0001 C CNN
-	1    7100 2300
-	0    1    1    0
-$EndComp
-Wire Wire Line
-	7150 2600 7200 2600
-Wire Wire Line
-	7200 2500 7150 2500
-Wire Wire Line
-	7150 2500 7150 2600
-Wire Wire Line
-	7100 2600 7150 2600
-Connection ~ 7150 2600
-Wire Wire Line
-	7150 2300 7150 2400
-Wire Wire Line
-	7150 2400 7200 2400
-Wire Wire Line
-	7100 2300 7150 2300
-Connection ~ 7150 2300
-Wire Wire Line
-	7150 2300 7200 2300
 Text Label 3000 3250 0    50   ~ 0
 I2S_LRCLK

Commit message: Clean up schematic for BoM export
- Change 22u 0805's (amp decoupling) to 15u
- Change 680n 0805's (part of output filter) to 470n
- Change C1 (amp bulk cap) from 820u to 1000u
- Add BoM.ini for KiBom export and
- Complete fields needed for KiBom (Manufacturer and partnumber)
Parts:
- C1: value 820u -> 1000u; Manufacturer (none) -> Nichicon; Partnumber (none) -> UHV1V102MHD
- J1: Manufacturer (none) -> JST; Partnumber (none) -> B3B-PH-K-S(LF)(SN)
- J4: Function Amp out / power in -> Power in / Amp out; Manufacturer (none) -> Dibo; Partnumber (none) -> DB128V-5.0-12P
- R7: Manufacturer (none) -> Yageo; Partnumber (none) -> RC0603FR-071KL
Changed lines of the file:
@@
 AR Path="/60B7AC16/60CBE8D5" Ref="C?"  Part="1"
 F 0 "C1" H 5900 5500 50  0000 L CNN
-F 1 "820u" H 5850 5400 50  0000 L CNN
+F 1 "1000u" H 5850 5400 50  0000 L CNN
 F 2 "ZOUDIO-footprints:Cap_Rad_D10_P5_horizontal" H 5838 5350 50  0001 C CNN
 F 3 "~" H 5800 5500 50  0001 C CNN
+F 4 "Nichicon" H 5800 5500 50  0001 C CNN "Manufacturer"
+F 5 "UHV1V102MHD" H 5800 5500 50  0001 C CNN "Partnumber"
 	1    5800 5500
 	1    0    0    -1
@@
 F 2 "Resistor_SMD:R_0603_1608Metric" H 5250 2350 50  0001 C CNN
 F 3 "~" H 5250 2350 50  0001 C CNN
+F 4 "Yageo" H 5250 2350 50  0001 C CNN "Manufacturer"
+F 5 "RC0603FR-071KL" H 5250 2350 50  0001 C CNN "Partnumber"
 	1    5250 2350
 	0    1    1    0
@@
 F 2 "ZOUDIO-footprints:Multicomp_12P_5mm" H 7400 3500 50  0001 C CNN
 F 3 "~" H 7400 3500 50  0001 C CNN
-F 4 "Amp out / power in" H 7900 3500 50  0000 C CNN "Function"
+F 4 "Power in / Amp out" H 7900 3500 50  0000 C CNN "Function"
+F 5 "Dibo" H 7400 3500 50  0001 C CNN "Manufacturer"
+F 6 "DB128V-5.0-12P" H 7400 3500 50  0001 C CNN "Partnumber"
 	1    7400 3500
 	1    0    0    1
@@
 F 3 "~" H 2800 3150 50  0001 C CNN
 F 4 "I2S" H 2950 3050 50  0000 C CNN "Function"
+F 5 "JST" H 2800 3150 50  0001 C CNN "Manufacturer"
+F 6 "B3B-PH-K-S(LF)(SN)" H 2800 3150 50  0001 C CNN "Partnumber"
 	1    2800 3150
 	-1   0    0    -1
