File: Mainboard/Microcontroller.sch (KiCad schematic (older format))
At the start: 17 parts, among them J3 PinHeader 02x03, J7 PinHeader 01x06, Q2 N-channel, U6 ATmega328PB-AU, U7 M24256 EEPROM, Y1 8MHz

Commit message: Modify library references
As described in the README of the newly added libraries submodule.
Schematic and PCB are synced.

Hardware folder is renamed to mainboard
Any other PCBs can be put in their own subfolder in the gitrepo

Commit also swaps source/drain of Q1 because it appeared wrong for some
reason after updating all symbol/footprints.
Parts:
- U7: symbol ZOUDIOsymbols:EEPROM_TSSOP -> ZOUDIO-symbols:EEPROM_TSSOP
Changed lines of the file:
@@
 	3550 5400 3550 5450
 $Comp
-L ZOUDIOsymbols:EEPROM_TSSOP U?
+L ZOUDIO-symbols:EEPROM_TSSOP U?
 U 1 1 5FD14DC1
 P 7050 2450

Commit message: Before testing CH340B and VCHG
Cleaned up amp lay-out a bit in the meanwhile
Parts:
- added C60: 100n, Capacitor_SMD:C_0603_1608Metric, symbol Device:C_Small
- C17, C54: Manufacturer Walsin -> Murata; Partnumber 0603B104J500CT -> GCM188L81H104KA57D
- J3: Config DNP -> dnp
- J7: value PinHeader 01x06 -> JST-PH 01x08; footprint Connector_JST:JST_PH_B6B-PH-K_1x06_P2.00mm_Vertical -> Connector_JST:JST_PH_B8B-PH-K_1x08_P2.00mm_Vertical; symbol Connector_Generic:Conn_01x06 -> Connector_Generic:Conn_01x08; Config DNP -> dnp
- R2, R4: value 10k -> 1k
Connections:
- net +5V is gone; now on net +3V3: J7.3 (Pin_3)
- net +3V3: now also C60.1; no longer J7.4 (Pin_4)
- net DTR: now also J7.6 (Pin_6)
- net GND: now also C60.2
- net I2C_SCL: now also J7.5 (Pin_5); no longer J7.6 (Pin_6)
- net I2C_SDA: now also J7.4 (Pin_4); no longer J7.5 (Pin_5)
- net UART_RX: now also J7.7 (Pin_7)
- net UART_TX: now also J7.8 (Pin_8)
Other:
- moved on the sheet: C34, C35, J3, Q2, R15, Y1

Commit message: Result after weekend of lay-out
Pretty far, just neats to be cleaned up for production.
Does not pass DRC yet.
Connections:
- net DTR: no longer J7.6 (Pin_6)
- net I2C_SCL: now also J7.8 (Pin_8); no longer J7.5 (Pin_5)
- net I2C_SDA: now also J7.7 (Pin_7); no longer J7.4 (Pin_4)
- net RESET: now also J7.6 (Pin_6)
- net UART_RX: now also J7.5 (Pin_5); no longer J7.7 (Pin_7)
- net UART_TX: now also J7.4 (Pin_4); no longer J7.8 (Pin_8)
Changed lines of the file:
@@
 	1    0    0    -1
 $EndComp
-Text Label 7900 5050 2    50   ~ 0
+Text Label 7900 5350 2    50   ~ 0
 I2C_SCL
-Text Label 7900 4950 2    50   ~ 0
+Text Label 7900 5250 2    50   ~ 0
 I2C_SDA
 Wire Wire Line
 	7000 4750 7900 4750
-Text Label 7900 5250 2    50   ~ 0
+Text Label 7900 5050 2    50   ~ 0
 UART_RX
-Text Label 7900 5350 2    50   ~ 0
+Text Label 7900 4950 2    50   ~ 0
 UART_TX
-Text Label 7900 5150 2    50   ~ 0
-DTR
 $Comp
 L Device:C_Small C?
@@
 Wire Wire Line
 	7700 2250 7750 2250
+Text Label 7900 5150 2    50   ~ 0
+RESET
 $EndSCHEMATC

Commit message: Mainboard: Version 1.0
Still need to clean up 3D models and BoM list,
but gerberexport-ready and ready to order.
Parts:
- added R52, R53, R54: 1k, Resistor_SMD:R_0603_1608Metric, symbol Device:R_Small
Connections:
- net PC1: now also Q2.1 (G), R15.1
- net PE1: no longer Q2.1 (G), R15.1
- net RESET: now also R53.1; no longer J7.6 (Pin_6)
- net UART_RX: now also R52.1; no longer J7.5 (Pin_5)
- net UART_TX: now also R54.1; no longer J7.4 (Pin_4)
- new net: J7.4 (Pin_4), R54.2
- new net: J7.5 (Pin_5), R52.2
- new net: J7.6 (Pin_6), R53.2
Other:
- moved on the sheet: J7, Q2, R15
Changed lines of the file:
@@
 Sheet 11 11
 Title "4x38W amp with DSP and BT"
-Date "2021-11-19"
-Rev "0.2"
+Date "2021-12-01"
+Rev "1.0"
 Comp "ZOUDIO"
 Comment1 ""
@@
 Text HLabel 4150 4700 2    50   Output ~ 0
 PD3
-Text HLabel 4150 3700 2    50   Output ~ 0
-PC1
 $Comp
 L Device:R_Small R?
@@
 	6300 2900 6300 1950
 Wire Notes Line
-	6300 4400 8950 4400
-Wire Notes Line
-	8950 4400 8950 5550
-Wire Notes Line
-	8950 5550 6300 5550
+	6300 4400 9550 4400
+Wire Notes Line
+	9550 4400 9550 5550
+Wire Notes Line
+	9550 5550 6300 5550
 Wire Notes Line
 	6300 5550 6300 4400
@@
 Expansion header
 Wire Wire Line
-	6650 5250 6650 5300
+	6600 5250 6600 5300
 $Comp
 L Device:R_Small R?
 U 1 1 5FC31722
-P 6650 5150
+P 6600 5150
 AR Path="/5FBDE745/5FC31722" Ref="R?"  Part="1"
 AR Path="/5FBDE62F/5FC31722" Ref="R?"  Part="1"
 AR Path="/60BB64C6/5FC31722" Ref="R15"  Part="1"
-F 0 "R15" H 6450 5200 50  0000 L CNN
-F 1 "10k" H 6450 5100 50  0000 L CNN
-F 2 "Resistor_SMD:R_0603_1608Metric" H 6650 5150 50  0001 C CNN
-F 3 "~" H 6650 5150 50  0001 C CNN
-F 4 "Uni-royal" H 6650 5150 50  0001 C CNN "Manufacturer"
-F 5 "0603WAF1002T5E" H 6650 5150 50  0001 C CNN "Partnumber"
-	1    6650 5150
+F 0 "R15" H 6400 5200 50  0000 L CNN
+F 1 "10k" H 6400 5100 50  0000 L CNN
+F 2 "Resistor_SMD:R_0603_1608Metric" H 6600 5150 50  0001 C CNN
+F 3 "~" H 6600 5150 50  0001 C CNN
+F 4 "Uni-royal" H 6600 5150 50  0001 C CNN "Manufacturer"
+F 5 "0603WAF1002T5E" H 6600 5150 50  0001 C CNN "Partnumber"
+	1    6600 5150
 	1    0    0    -1
 $EndComp
@@
 L power:VDD #PWR?
 U 1 1 5FC1F0F7
-P 7850 4650
+P 8550 4650
 AR Path="/5FC1F0F7" Ref="#PWR?"  Part="1"
 AR Path="/5FBDE62F/5FC1F0F7" Ref="#PWR?"  Part="1"
 AR Path="/60BB64C6/5FC1F0F7" Ref="#PWR0154"  Part="1"
-F 0 "#PWR0154" H 7850 4500 50  0001 C CNN
-F 1 "VDD" V 7850 4850 50  0000 C CNN
-F 2 "" H 7850 4650 50  0001 C CNN
-F 3 "" H 7850 4650 50  0001 C CNN
-	1    7850 4650
+F 0 "#PWR0154" H 8550 4500 50  0001 C CNN
+F 1 "VDD" V 8550 4850 50  0000 C CNN
+F 2 "" H 8550 4650 50  0001 C CNN
+F 3 "" H 8550 4650 50  0001 C CNN
+	1    8550 4650
 	0    -1   -1   0
 $EndComp
@@
 L power:+3V3 #PWR?
 U 1 1 5FC1F0F1
-P 7850 4850
+P 8550 4850
 AR Path="/5FC1F0F1" Ref="#PWR?"  Part="1"
 AR Path="/5FBDE62F/5FC1F0F1" Ref="#PWR?"  Part="1"
 AR Path="/60BB64C6/5FC1F0F1" Ref="#PWR0155"  Part="1"
-F 0 "#PWR0155" H 7850 4700 50  0001 C CNN
-F 1 "+3V3" V 7850 5050 50  0000 C CNN
-F 2 "" H 7850 4850 50  0001 C CNN
-F 3 "" H 7850 4850 50  0001 C CNN
-	1    7850 4850
+F 0 "#PWR0155" H 8550 4700 50  0001 C CNN
+F 1 "+3V3" V 8550 5050 50  0000 C CNN
+F 2 "" H 8550 4850 50  0001 C CNN
+F 3 "" H 8550 4850 50  0001 C CNN
+	1    8550 4850
 	0    -1   -1   0
 $EndComp
@@
 L Connector_Generic:Conn_01x08 J7
 U 1 1 5FBE811C
-P 8100 4950
-F 0 "J7" H 8200 5050 50  0000 L CNN
-F 1 "JST-PH 01x08" H 8200 4950 50  0000 L CNN
-F 2 "Connector_JST:JST_PH_B8B-PH-K_1x08_P2.00mm_Vertical" H 8100 4950 50  0001 C CNN
-F 3 "~" H 8100 4950 50  0001 C CNN
-F 4 "Expansion" H 8400 4850 50  0000 C CNN "Function"
-F 5 "dnp" H 8300 4750 50  0000 C CNN "Config"
-	1    8100 4950
+P 8800 4950
+F 0 "J7" H 8900 5050 50  0000 L CNN
+F 1 "JST-PH 01x08" H 8900 4950 50  0000 L CNN
+F 2 "Connector_JST:JST_PH_B8B-PH-K_1x08_P2.00mm_Vertical" H 8800 4950 50  0001 C CNN
+F 3 "~" H 8800 4950 50  0001 C CNN
+F 4 "Expansion" H 9100 4850 50  0000 C CNN "Function"
+F 5 "dnp" H 9000 4750 50  0000 C CNN "Config"
+	1    8800 4950
 	1    0    0    -1
 $EndComp
@@
 L Device:Q_NMOS_GSD Q2
 U 1 1 61058F11
-P 6900 5000
-F 0 "Q2" H 7200 5050 50  0000 C CNN
-F 1 "N-channel" H 7300 4950 50  0000 C CNN
-F 2 "Package_TO_SOT_SMD:SOT-23" H 7100 5100 50  0001 C CNN
-F 3 "~" H 6900 5000 50  0001 C CNN
-	1    6900 5000
-	1    0    0    -1
-$EndComp
-Wire Wire Line
-	7850 4650 7900 4650
-Wire Wire Line
-	7900 4850 7850 4850
+P 6850 5000
+F 0 "Q2" H 7150 5050 50  0000 C CNN
+F 1 "N-channel" H 7250 4950 50  0000 C CNN
+F 2 "Package_TO_SOT_SMD:SOT-23" H 7050 5100 50  0001 C CNN
+F 3 "~" H 6850 5000 50  0001 C CNN
+	1    6850 5000
+	1    0    0    -1
+$EndComp
+Wire Wire Line
+	8550 4650 8600 4650
+Wire Wire Line
+	8600 4850 8550 4850
 $Comp
 L Device:R_Small R?
@@
 L power:GND #PWR0163
 U 1 1 61CDF06B
-P 6650 5300
-F 0 "#PWR0163" H 6650 5050 50  0001 C CNN
-F 1 "GND" H 6650 5150 50  0000 C CNN
-F 2 "" H 6650 5300 50  0001 C CNN
-F 3 "" H 6650 5300 50  0001 C CNN
-	1    6650 5300
+P 6600 5300
+F 0 "#PWR0163" H 6600 5050 50  0001 C CNN
+F 1 "GND" H 6600 5150 50  0000 C CNN
+F 2 "" H 6600 5300 50  0001 C CNN
+F 3 "" H 6600 5300 50  0001 C CNN
+	1    6600 5300
 	1    0    0    -1
 $EndComp
@@
 L power:GND #PWR0164
 U 1 1 61CE0960
-P 7000 5300
-F 0 "#PWR0164" H 7000 5050 50  0001 C CNN
-F 1 "GND" H 7000 5150 50  0000 C CNN
-F 2 "" H 7000 5300 50  0001 C CNN
-F 3 "" H 7000 5300 50  0001 C CNN
-	1    7000 5300
-	1    0    0    -1
-$EndComp
-Wire Wire Line
-	7000 4800 7000 4750
-Wire Wire Line
-	7000 5200 7000 5300
-Wire Wire Line
-	6650 5050 6650 5000
+P 6950 5300
+F 0 "#PWR0164" H 6950 5050 50  0001 C CNN
+F 1 "GND" H 6950 5150 50  0000 C CNN
+F 2 "" H 6950 5300 50  0001 C CNN
+F 3 "" H 6950 5300 50  0001 C CNN
+	1    6950 5300
+	1    0    0    -1
+$EndComp
+Wire Wire Line
+	6950 4800 6950 4750
+Wire Wire Line
+	6950 5200 6950 5300
+Wire Wire Line
+	6600 5050 6600 5000
+Wire Wire Line
+	6550 5000 6600 5000
+Connection ~ 6600 5000
 Wire Wire Line
 	6600 5000 6650 5000
-Connection ~ 6650 5000
-Wire Wire Line
-	6650 5000 6700 5000
-Text Label 6600 5000 2    50   ~ 0
-PE1
 $Comp
 L power:GND #PWR0165
@@
 	1    0    0    -1
 $EndComp
-Text Label 7900 5350 2    50   ~ 0
+Text Label 8600 5350 2    50   ~ 0
 I2C_SCL
-Text Label 7900 5250 2    50   ~ 0
+Text Label 8600 5250 2    50   ~ 0
 I2C_SDA
 Wire Wire Line
-	7000 4750 7900 4750
-Text Label 7900 5050 2    50   ~ 0
+	6950 4750 8600 4750
+Text Label 7900 5100 2    50   ~ 0
 UART_RX
 Text Label 7900 4950 2    50   ~ 0
@@
 Wire Wire Line
 	7700 2250 7750 2250
-Text Label 7900 5150 2    50   ~ 0
+Text Label 7900 5250 2    50   ~ 0
 RESET
+$Comp
+L Device:R_Small R?
+U 1 1 61A67700
+P 8050 4950
+AR Path="/61A67700" Ref="R?"  Part="1"
+AR Path="/5FCC1D27/61A67700" Ref="R?"  Part="1"
+AR Path="/5FBDE62F/61A67700" Ref="R?"  Part="1"
+AR Path="/60BB64C6/61A67700" Ref="R54"  Part="1"
+F 0 "R54" V 8150 4950 50  0000 L BNN
+F 1 "1k" V 8150 4800 50  0000 L BNN
+F 2 "Resistor_SMD:R_0603_1608Metric" H 8050 4950 50  0001 C CNN
+F 3 "~" H 8050 4950 50  0001 C CNN
+F 4 "Uni-royal" H 8050 4950 50  0001 C CNN "Manufacturer"
+F 5 "0603WAF1002T5E" H 8050 4950 50  0001 C CNN "Partnumber"
+	1    8050 4950
+	0    -1   -1   0
+$EndComp
+$Comp
+L Device:R_Small R?
+U 1 1 61A68600
+P 8050 5100
+AR Path="/61A68600" Ref="R?"  Part="1"
+AR Path="/5FCC1D27/61A68600" Ref="R?"  Part="1"
+AR Path="/5FBDE62F/61A68600" Ref="R?"  Part="1"
+AR Path="/60BB64C6/61A68600" Ref="R52"  Part="1"
+F 0 "R52" V 8150 5100 50  0000 L BNN
+F 1 "1k" V 8150 4950 50  0000 L BNN
+F 2 "Resistor_SMD:R_0603_1608Metric" H 8050 5100 50  0001 C CNN
+F 3 "~" H 8050 5100 50  0001 C CNN
+F 4 "Uni-royal" H 8050 5100 50  0001 C CNN "Manufacturer"
+F 5 "0603WAF1002T5E" H 8050 5100 50  0001 C CNN "Partnumber"
+	1    8050 5100
+	0    -1   -1   0
+$EndComp
+$Comp
+L Device:R_Small R?
+U 1 1 61A68AA2
+P 8050 5250
+AR Path="/61A68AA2" Ref="R?"  Part="1"
+AR Path="/5FCC1D27/61A68AA2" Ref="R?"  Part="1"
+AR Path="/5FBDE62F/61A68AA2" Ref="R?"  Part="1"
+AR Path="/60BB64C6/61A68AA2" Ref="R53"  Part="1"
+F 0 "R53" V 8150 5250 50  0000 L BNN
+F 1 "1k" V 8150 5100 50  0000 L BNN
+F 2 "Resistor_SMD:R_0603_1608Metric" H 8050 5250 50  0001 C CNN
+F 3 "~" H 8050 5250 50  0001 C CNN
+F 4 "Uni-royal" H 8050 5250 50  0001 C CNN "Manufacturer"
+F 5 "0603WAF1002T5E" H 8050 5250 50  0001 C CNN "Partnumber"
+	1    8050 5250
+	0    -1   -1   0
+$EndComp
+Wire Wire Line
+	8150 4950 8600 4950
+Wire Wire Line
+	8600 5050 8250 5050
+Wire Wire Line
+	8250 5050 8250 5100
+Wire Wire Line
+	8250 5100 8150 5100
+Wire Wire Line
+	8600 5150 8250 5150
+Wire Wire Line
+	8250 5150 8250 5250
+Wire Wire Line
+	8250 5250 8150 5250
+Wire Wire Line
+	7900 5250 7950 5250
+Wire Wire Line
+	7900 5100 7950 5100
+Wire Wire Line
+	7900 4950 7950 4950
+Text Label 4150 3700 0    50   ~ 0
+PC1
+Text Label 6550 5000 2    50   ~ 0
+PC1
 $EndSCHEMATC

Commit message: Clean up schematic for BoM export
- Change 22u 0805's (amp decoupling) to 15u
- Change 680n 0805's (part of output filter) to 470n
- Change C1 (amp bulk cap) from 820u to 1000u
- Add BoM.ini for KiBom export and
- Complete fields needed for KiBom (Manufacturer and partnumber)
Parts:
- J7: Config dnp -> (none); Manufacturer (none) -> JST; Partnumber (none) -> B8B-PH-K-S(LF)(SN)
- Q2: Manufacturer (none) -> Vishay; Partnumber (none) -> SI2316BDS-T1-GE3
- R11, R12, R13, R14, R15: Manufacturer Uni-royal -> Yageo; Partnumber 0603WAF1002T5E -> RC0603FR-0710KL
- R2, R4, R52, R53, R54: Manufacturer Uni-royal -> Yageo; Partnumber 0603WAF1002T5E -> RC0603FR-071KL
- U6: value ATmega328PB-AU -> ATMEGA328PB-AU; Manufacturer (none) -> Microchip; Partnumber (none) -> ATMEGA328PB-AU
- Y1: Manufacturer (none) -> ECS; Partnumber (none) -> ECS-80-18-30B-AGN-TR
Changed lines of the file:
@@
 F 2 "Resistor_SMD:R_0603_1608Metric" H 4650 3850 50  0001 C CNN
 F 3 "~" H 4650 3850 50  0001 C CNN
-F 4 "Uni-royal" H 4650 3850 50  0001 C CNN "Manufacturer"
-F 5 "0603WAF1002T5E" H 4650 3850 50  0001 C CNN "Partnumber"
+F 4 "Yageo" H 4650 3850 50  0001 C CNN "Manufacturer"
+F 5 "RC0603FR-071KL" H 4650 3850 50  0001 C CNN "Partnumber"
 	1    4650 3850
 	1    0    0    -1
@@
 F 2 "Resistor_SMD:R_0603_1608Metric" H 4900 3850 50  0001 C CNN
 F 3 "~" H 4900 3850 50  0001 C CNN
-F 4 "Uni-royal" H 4900 3850 50  0001 C CNN "Manufacturer"
-F 5 "0603WAF1002T5E" H 4900 3850 50  0001 C CNN "Partnumber"
+F 4 "Yageo" H 4900 3850 50  0001 C CNN "Manufacturer"
+F 5 "RC0603FR-071KL" H 4900 3850 50  0001 C CNN "Partnumber"
 	1    4900 3850
 	1    0    0    -1
@@
 F 2 "Resistor_SMD:R_0603_1608Metric" H 4800 3300 50  0001 C CNN
 F 3 "~" H 4800 3300 50  0001 C CNN
-F 4 "Uni-royal" H 4800 3300 50  0001 C CNN "Manufacturer"
-F 5 "0603WAF1002T5E" H 4800 3300 50  0001 C CNN "Partnumber"
+F 4 "Yageo" H 4800 3300 50  0001 C CNN "Manufacturer"
+F 5 "RC0603FR-0710KL" H 4800 3300 50  0001 C CNN "Partnumber"
 	1    4800 3300
 	0    1    1    0
@@
 F 2 "Resistor_SMD:R_0603_1608Metric" H 5500 4000 50  0001 C CNN
 F 3 "~" H 5500 4000 50  0001 C CNN
-F 4 "Uni-royal" H 5500 4000 50  0001 C CNN "Manufacturer"
-F 5 "0603WAF1002T5E" H 5500 4000 50  0001 C CNN "Partnumber"
+F 4 "Yageo" H 5500 4000 50  0001 C CNN "Manufacturer"
+F 5 "RC0603FR-0710KL" H 5500 4000 50  0001 C CNN "Partnumber"
 	1    5500 4000
 	-1   0    0    1
@@
 F 2 "Resistor_SMD:R_0603_1608Metric" H 6600 5150 50  0001 C CNN
 F 3 "~" H 6600 5150 50  0001 C CNN
-F 4 "Uni-royal" H 6600 5150 50  0001 C CNN "Manufacturer"
-F 5 "0603WAF1002T5E" H 6600 5150 50  0001 C CNN "Partnumber"
+F 4 "Yageo" H 6600 5150 50  0001 C CNN "Manufacturer"
+F 5 "RC0603FR-0710KL" H 6600 5150 50  0001 C CNN "Partnumber"
 	1    6600 5150
 	1    0    0    -1
@@
 F 3 "~" H 8800 4950 50  0001 C CNN
 F 4 "Expansion" H 9100 4850 50  0000 C CNN "Function"
-F 5 "dnp" H 9000 4750 50  0000 C CNN "Config"
+F 5 "" H 9000 4750 50  0000 C CNN "Config"
+F 6 "JST" H 8800 4950 50  0001 C CNN "Manufacturer"
+F 7 "B8B-PH-K-S(LF)(SN)" H 8800 4950 50  0001 C CNN "Partnumber"
 	1    8800 4950
 	1    0    0    -1
@@
 F 2 "Crystal:Crystal_SMD_Abracon_ABM3C-4Pin_5.0x3.2mm" H 8950 2450 50  0001 C CNN
 F 3 "~" H 8950 2450 50  0001 C CNN
+F 4 "ECS" H 8950 2450 50  0001 C CNN "Manufacturer"
+F 5 "ECS-80-18-30B-AGN-TR" H 8950 2450 50  0001 C CNN "Partnumber"
 	1    8950 2450
 	-1   0    0    1
@@
 P 3550 3900
 F 0 "U6" H 3450 4050 50  0000 C CNN
-F 1 "ATmega328PB-AU" H 3450 3950 50  0000 C CNN
+F 1 "ATMEGA328PB-AU" H 3450 3950 50  0000 C CNN
 F 2 "Package_QFP:TQFP-32_7x7mm_P0.8mm" H 3550 3900 50  0001 C CIN
 F 3 "~" H 3550 3900 50  0001 C CNN
+F 4 "Microchip" H 3550 3900 50  0001 C CNN "Manufacturer"
+F 5 "ATMEGA328PB-AU" H 3550 3900 50  0001 C CNN "Partnumber"
 	1    3550 3900
 	1    0    0    -1
@@
 F 2 "Package_TO_SOT_SMD:SOT-23" H 7050 5100 50  0001 C CNN
 F 3 "~" H 6850 5000 50  0001 C CNN
+F 4 "Vishay" H 6850 5000 50  0001 C CNN "Manufacturer"
+F 5 "SI2316BDS-T1-GE3" H 6850 5000 50  0001 C CNN "Partnumber"
 	1    6850 5000
 	1    0    0    -1
@@
 F 2 "Resistor_SMD:R_0603_1608Metric" H 4800 3100 50  0001 C CNN
 F 3 "~" H 4800 3100 50  0001 C CNN
-F 4 "Uni-royal" H 4800 3100 50  0001 C CNN "Manufacturer"
-F 5 "0603WAF1002T5E" H 4800 3100 50  0001 C CNN "Partnumber"
+F 4 "Yageo" H 4800 3100 50  0001 C CNN "Manufacturer"
+F 5 "RC0603FR-0710KL" H 4800 3100 50  0001 C CNN "Partnumber"
 	1    4800 3100
 	0    1    1    0
@@
 F 2 "Resistor_SMD:R_0603_1608Metric" H 4800 2900 50  0001 C CNN
 F 3 "~" H 4800 2900 50  0001 C CNN
-F 4 "Uni-royal" H 4800 2900 50  0001 C CNN "Manufacturer"
-F 5 "0603WAF1002T5E" H 4800 2900 50  0001 C CNN "Partnumber"
+F 4 "Yageo" H 4800 2900 50  0001 C CNN "Manufacturer"
+F 5 "RC0603FR-0710KL" H 4800 2900 50  0001 C CNN "Partnumber"
 	1    4800 2900
 	0    1    1    0
@@
 F 2 "Resistor_SMD:R_0603_1608Metric" H 8050 4950 50  0001 C CNN
 F 3 "~" H 8050 4950 50  0001 C CNN
-F 4 "Uni-royal" H 8050 4950 50  0001 C CNN "Manufacturer"
-F 5 "0603WAF1002T5E" H 8050 4950 50  0001 C CNN "Partnumber"
+F 4 "Yageo" H 8050 4950 50  0001 C CNN "Manufacturer"
+F 5 "RC0603FR-071KL" H 8050 4950 50  0001 C CNN "Partnumber"
 	1    8050 4950
 	0    -1   -1   0
@@
 F 2 "Resistor_SMD:R_0603_1608Metric" H 8050 5100 50  0001 C CNN
 F 3 "~" H 8050 5100 50  0001 C CNN
-F 4 "Uni-royal" H 8050 5100 50  0001 C CNN "Manufacturer"
-F 5 "0603WAF1002T5E" H 8050 5100 50  0001 C CNN "Partnumber"
+F 4 "Yageo" H 8050 5100 50  0001 C CNN "Manufacturer"
+F 5 "RC0603FR-071KL" H 8050 5100 50  0001 C CNN "Partnumber"
 	1    8050 5100
 	0    -1   -1   0
@@
 F 2 "Resistor_SMD:R_0603_1608Metric" H 8050 5250 50  0001 C CNN
 F 3 "~" H 8050 5250 50  0001 C CNN
-F 4 "Uni-royal" H 8050 5250 50  0001 C CNN "Manufacturer"
-F 5 "0603WAF1002T5E" H 8050 5250 50  0001 C CNN "Partnumber"
+F 4 "Yageo" H 8050 5250 50  0001 C CNN "Manufacturer"
+F 5 "RC0603FR-071KL" H 8050 5250 50  0001 C CNN "Partnumber"
 	1    8050 5250
 	0    -1   -1   0
