File: Mainboard/User-controls.sch (KiCad schematic (older format))
At the start: 11 parts, among them J2 JST-PH 01x10, J5 JST-PH 01x02, J6 JST-PH 01x02

Commit message: Clean up schematic for BoM export
- Change 22u 0805's (amp decoupling) to 15u
- Change 680n 0805's (part of output filter) to 470n
- Change C1 (amp bulk cap) from 820u to 1000u
- Add BoM.ini for KiBom export and
- Complete fields needed for KiBom (Manufacturer and partnumber)
Parts:
- J2: Manufacturer (none) -> JST; Partnumber (none) -> B10B-PH-K-S(LF)(SN)
- J5, J6: Manufacturer (none) -> JST; Partnumber (none) -> B2B-PH-K-S(LF)(SN)
- R22, R23, R25: Manufacturer (none) -> Yageo; Partnumber (none) -> RC0603FR-07100KL
- R24: Manufacturer (none) -> Yageo; Partnumber (none) -> RC0603FR-071KL
- R35, R36, R38, R39: Manufacturer Uni-royal -> Yageo; Partnumber 0603WAF1001T5E -> RC0603FR-071KL
Changed lines of the file:
@@
 F 2 "Resistor_SMD:R_0603_1608Metric" H 5550 2250 50  0001 C CNN
 F 3 "~" H 5550 2250 50  0001 C CNN
+F 4 "Yageo" H 5550 2250 50  0001 C CNN "Manufacturer"
+F 5 "RC0603FR-07100KL" H 5550 2250 50  0001 C CNN "Partnumber"
 	1    5550 2250
 	1    0    0    -1
@@
 F 3 "~" H 5300 2000 50  0001 C CNN
 F 4 "TrueWirelessStereo switch" H 5400 1850 50  0000 L CNN "Function"
+F 5 "JST" H 5300 2000 50  0001 C CNN "Manufacturer"
+F 6 "B2B-PH-K-S(LF)(SN)" H 5300 2000 50  0001 C CNN "Partnumber"
 	1    5300 2000
 	-1   0    0    -1
@@
 F 3 "~" H 5300 4100 50  0001 C CNN
 F 4 "Main control" H 5400 3950 50  0000 L CNN "Function"
+F 5 "JST" H 5300 4100 50  0001 C CNN "Manufacturer"
+F 6 "B10B-PH-K-S(LF)(SN)" H 5300 4100 50  0001 C CNN "Partnumber"
 	1    5300 4100
 	-1   0    0    -1
@@
 F 2 "Resistor_SMD:R_0603_1608Metric" H 5650 3700 50  0001 C CNN
 F 3 "~" H 5650 3700 50  0001 C CNN
+F 4 "Yageo" H 5650 3700 50  0001 C CNN "Manufacturer"
+F 5 "RC0603FR-071KL" H 5650 3700 50  0001 C CNN "Partnumber"
 	1    5650 3700
 	0    -1   -1   0
@@
 F 3 "~" H 5300 2750 50  0001 C CNN
 F 4 "EQ switch" H 5400 2600 50  0000 L CNN "Function"
+F 5 "JST" H 5300 2750 50  0001 C CNN "Manufacturer"
+F 6 "B2B-PH-K-S(LF)(SN)" H 5300 2750 50  0001 C CNN "Partnumber"
 	1    5300 2750
 	-1   0    0    -1
@@
 F 2 "Resistor_SMD:R_0603_1608Metric" H 5550 3000 50  0001 C CNN
 F 3 "~" H 5550 3000 50  0001 C CNN
+F 4 "Yageo" H 5550 3000 50  0001 C CNN "Manufacturer"
+F 5 "RC0603FR-07100KL" H 5550 3000 50  0001 C CNN "Partnumber"
 	1    5550 3000
 	1    0    0    -1
@@
 F 2 "Resistor_SMD:R_0603_1608Metric" H 6050 5700 50  0001 C CNN
 F 3 "~" H 6050 5700 50  0001 C CNN
-F 4 "Uni-royal" H 6050 5700 50  0001 C CNN "Manufacturer"
-F 5 "0603WAF1001T5E" H 6050 5700 50  0001 C CNN "Partnumber"
+F 4 "Yageo" H 6050 5700 50  0001 C CNN "Manufacturer"
+F 5 "RC0603FR-071KL" H 6050 5700 50  0001 C CNN "Partnumber"
 	1    6050 5700
 	0    1    1    0
@@
 F 2 "Resistor_SMD:R_0603_1608Metric" H 6200 5850 50  0001 C CNN
 F 3 "~" H 6200 5850 50  0001 C CNN
-F 4 "Uni-royal" H 6200 5850 50  0001 C CNN "Manufacturer"
-F 5 "0603WAF1001T5E" H 6200 5850 50  0001 C CNN "Partnumber"
+F 4 "Yageo" H 6200 5850 50  0001 C CNN "Manufacturer"
+F 5 "RC0603FR-071KL" H 6200 5850 50  0001 C CNN "Partnumber"
 	1    6200 5850
 	-1   0    0    1
@@
 F 2 "Resistor_SMD:R_0603_1608Metric" H 6050 4900 50  0001 C CNN
 F 3 "~" H 6050 4900 50  0001 C CNN
-F 4 "Uni-royal" H 6050 4900 50  0001 C CNN "Manufacturer"
-F 5 "0603WAF1001T5E" H 6050 4900 50  0001 C CNN "Partnumber"
+F 4 "Yageo" H 6050 4900 50  0001 C CNN "Manufacturer"
+F 5 "RC0603FR-071KL" H 6050 4900 50  0001 C CNN "Partnumber"
 	1    6050 4900
 	0    1    1    0
@@
 F 2 "Resistor_SMD:R_0603_1608Metric" H 6200 5050 50  0001 C CNN
 F 3 "~" H 6200 5050 50  0001 C CNN
-F 4 "Uni-royal" H 6200 5050 50  0001 C CNN "Manufacturer"
-F 5 "0603WAF1001T5E" H 6200 5050 50  0001 C CNN "Partnumber"
+F 4 "Yageo" H 6200 5050 50  0001 C CNN "Manufacturer"
+F 5 "RC0603FR-071KL" H 6200 5050 50  0001 C CNN "Partnumber"
 	1    6200 5050
 	-1   0    0    1
@@
 F 2 "Resistor_SMD:R_0603_1608Metric" H 6200 4350 50  0001 C CNN
 F 3 "~" H 6200 4350 50  0001 C CNN
+F 4 "Yageo" H 6200 4350 50  0001 C CNN "Manufacturer"
+F 5 "RC0603FR-07100KL" H 6200 4350 50  0001 C CNN "Partnumber"
 	1    6200 4350
 	-1   0    0    1
