File: Mainboard/AIO438.kicad_pcb (KiCad board)
At the start: 4 copper layers, 121 x 60 mm, 162 parts, among them J1 JST-PH 01x03, J10 U.FL, J11 JST-PH 01x02, J2 JST-PH 01x10, J3 PinHeader 02x03, J4 5mm screwterminal 01x12, J5 JST-PH 01x02, J6 JST-PH 01x02, J7 JST-PH 01x08, J8 USB-C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

Commit message: Mainboard: Version 1.0
Still need to clean up 3D models and BoM list,
but gerberexport-ready and ready to order.
Parts:
- removed TP5: TestPoint, TestPoint:TestPoint_Pad_D1.0mm
- added R52: 1k, Resistor_SMD:R_0603_1608Metric, F.Cu at (131.9, 125.9)
- added R53: 1k, Resistor_SMD:R_0603_1608Metric, F.Cu at (135.3, 125.9)
- added R54: 1k, Resistor_SMD:R_0603_1608Metric, F.Cu at (128.5, 125.9)
- LOGO1: footprint ZOUDIO-footprints:ZOUDIO25mm -> ZOUDIO-footprints:ZOUDIO25mm_mask
- U4: footprint Package_SON:WSON-10-1EP_2x3mm_P0.5mm_EP0.84x2.4mm_ThermalVias -> ZOUDIO-footprints:WSON-10-1EP_2x3mm_P0.5mm_EP0.84x2.4mm
- moved LOGO1 47.6 mm to (155.7, 89.0)
- moved R2 5.46 mm to (124.4, 114.1), turned to 90 degrees
- moved R4 5.46 mm to (122.8, 114.1), turned to 90 degrees
- moved C60 4.23 mm to (136.3, 113.6), turned to 270 degrees
- moved R6 3.96 mm to (121.3, 100.1)
- moved R5 3.96 mm to (122.9, 100.1)
- moved U7 3.55 mm to (131.4, 113.6)
- moved R14 0.82 mm to (122.8, 110.0)
- moved R12 0.50 mm to (177.7, 124.3)
- moved R25 0.50 mm to (177.7, 125.9)
- moved C39 0.36 mm to (182.0, 103.8)
- moved C18 0.32 mm to (172.8, 103.8)
- moved C53 0.32 mm to (183.9, 104.0)
- moved C59 0.32 mm to (168.8, 104.0)
- moved C41 0.30 mm to (170.9, 104.0)
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Connections:
- net /USB/I2C_SCL renamed Net-(U8-Pad22)
- net /USB/I2C_SDA renamed Net-(U8-Pad2)
- net /USB/LED2 renamed Net-(U8-Pad23)
- J7 pad 4: /USB to UART/UART_RX -> Net-(J7-Pad4)
- J7 pad 5: /Microcontroller/UART_RX -> Net-(J7-Pad5)
- J7 pad 6: /Microcontroller/RESET -> Net-(J7-Pad6)
- Q2 pad 1: /Power/Buck_sleep -> /Microcontroller/PC1
- R15 pad 1: /Power/Buck_sleep -> /Microcontroller/PC1
- U10 pad 25: /Microcontroller/PC1 -> Net-(U10-Pad25)
Routing:
- net /Microcontroller/PC1: track 88.7 -> 14.6 mm
- net VDD: track 0.83 -> 37.2 mm, vias 28 -> 32
- net /Power/Buck_sleep: track 53.2 -> 28.0 mm, vias 3 -> 0
- net 3V3_USB: track 123.4 -> 147.5 mm, vias 20 -> 22
- net /Microcontroller/PC3: track 0.00 -> 15.3 mm, vias 0 -> 2
- net /Amplifiers/I2C_SDA: track 99.2 -> 111.4 mm, vias 3 -> 5
- net /Amplifiers/I2C_SCL: track 98.6 -> 109.6 mm, vias 4 -> 6
- net /Power/3V3_buck: track 20.2 -> 26.4 mm
- net GND: track 36.3 -> 40.5 mm, vias 132 -> 165
- net Net-(J7-Pad6): track 0.00 -> 4.09 mm
- net Net-(J7-Pad4): track 0.00 -> 4.07 mm
- net +3V3: track 32.7 -> 36.3 mm, vias 25 -> 24
- net Net-(J7-Pad5): track 0.00 -> 3.51 mm
- net /USB to UART/UART_RX: track 115.5 -> 112.1 mm, vias 3 -> 5
- net /User controls/AUX_GND: track 78.0 -> 80.9 mm
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Other:
- board text added: "AIO438 www.ZOUDIO.com The Netherlands"
- board text added: "EQ SW"
- board text added: "HW V1.0"
- board text added: "Main"
- board text added: "TWS SW"
- board text removed: "AUX"
- board text removed: "EQ"
- board text removed: "LED"
- board text removed: "ROT"
- board text removed: "ZOUDIO AIO438 www.ZOUDIO.com The Netherlands"

Commit message: Update project to Kicad 6
Convert schematic and layout
Remove all other redundant files
Routing:
- added copper zone on In2.Cu, net +3V3
- added copper zone on In2.Cu, net 3V3_USB
- added copper zone on In1.Cu, net GND
- added copper zone on In2.Cu, net VDD
- removed copper zone on In2.PWR, net +3V3
- removed copper zone on In2.PWR, net 3V3_USB
- removed copper zone on In1.GND, net GND
- removed copper zone on In2.PWR, net VDD
Other:
- net class Default removed

Commit message: Update lay-out and fix legacy 3d models
Update lay-out from schematic
Add legacy 3d model searchpath KISYS3DMOD
Parts:
- C1: value 820u -> 1000u
- C12, C14, C15, C16, C30, C31, C32, C33: value 680n -> 470n
- C40, C41, C52, C53, C55, C56, C58, C59: value 22u -> 15u
- U4: value TPS62177DQC -> TPS62177
- U6: value ATmega328PB-AU -> ATMEGA328PB-AU
- U8: value FE1.1s-BQFN24B -> FE1.1S
Connections:
- net /Amplifiers/I2C_SCL renamed /Microcontroller/I2C_SCL
- net /Amplifiers/I2C_SDA renamed /Microcontroller/I2C_SDA
- net /Microcontroller/DTR renamed /USB to UART/UART_DTR
- net /Microcontroller/PB1 renamed /Bluetooth/PIO22
- net /Microcontroller/PB2 renamed /Bluetooth/PIO21
- net /Microcontroller/PE2 renamed /Bluetooth/PIO20
- net /Microcontroller/PE3 renamed /Bluetooth/PIO19
- net /Power/Buck_sleep renamed /Microcontroller/PE1
- net /USB to UART/UART_RX renamed /Microcontroller/UART_TX
- net /USB/D2+ renamed /Bluetooth/USB_DP
- net /USB/D2- renamed /Bluetooth/USB_DN
- net /User controls/AUX_GND renamed /Bluetooth/MIC_N
- net /User controls/AUX_L renamed /Bluetooth/MIC1_P
- net /User controls/AUX_R renamed /Bluetooth/MIC2_P
- net /User controls/EQ_SW renamed /Microcontroller/PB3
- net /User controls/LED_GREEN renamed /Microcontroller/PD5
- net /User controls/LED_RED renamed /Microcontroller/PD6
- J8 pad A8: Net-(J8-PadA8) -> unconnected-(J8-PadA8)
- J8 pad B8: Net-(J8-PadB8) -> unconnected-(J8-PadB8)
- U1 pad 10: Net-(U1-Pad10) -> unconnected-(U1-Pad10)
- U1 pad 11: Net-(U1-Pad11) -> unconnected-(U1-Pad11)
- U1 pad 9: Net-(U1-Pad9) -> unconnected-(U1-Pad9)
- U10 pad 1: Net-(U10-Pad1) -> unconnected-(U10-Pad1)
- U10 pad 12: Net-(U10-Pad12) -> unconnected-(U10-Pad12)
- U10 pad 19: Net-(U10-Pad19) -> unconnected-(U10-Pad19)
- U10 pad 22: Net-(U10-Pad22) -> unconnected-(U10-Pad22)
- U10 pad 25: Net-(U10-Pad25) -> unconnected-(U10-Pad25)
- U10 pad 26: Net-(U10-Pad26) -> unconnected-(U10-Pad26)
- U10 pad 27: Net-(U10-Pad27) -> unconnected-(U10-Pad27)
- U10 pad 28: Net-(U10-Pad28) -> unconnected-(U10-Pad28)
- U10 pad 29: Net-(U10-Pad29) -> unconnected-(U10-Pad29)
- U10 pad 30: Net-(U10-Pad30) -> unconnected-(U10-Pad30)
- U10 pad 31: Net-(U10-Pad31) -> unconnected-(U10-Pad31)
- U10 pad 32: Net-(U10-Pad32) -> unconnected-(U10-Pad32)
- U10 pad 33: Net-(U10-Pad33) -> unconnected-(U10-Pad33)
- U10 pad 34: Net-(U10-Pad34) -> unconnected-(U10-Pad34)
- U10 pad 35: Net-(U10-Pad35) -> unconnected-(U10-Pad35)
- U10 pad 36: Net-(U10-Pad36) -> unconnected-(U10-Pad36)
- U10 pad 37: Net-(U10-Pad37) -> unconnected-(U10-Pad37)
- U10 pad 39: Net-(U10-Pad39) -> unconnected-(U10-Pad39)
- U10 pad 48: Net-(U10-Pad48) -> unconnected-(U10-Pad48)
- U10 pad 49: Net-(U10-Pad49) -> unconnected-(U10-Pad49)
- U10 pad 50: Net-(U10-Pad50) -> unconnected-(U10-Pad50)
- U10 pad 51: Net-(U10-Pad51) -> unconnected-(U10-Pad51)
- U10 pad 6: Net-(U10-Pad6) -> unconnected-(U10-Pad6)
- U2 pad 10: Net-(U2-Pad10) -> unconnected-(U2-Pad10)
- U2 pad 11: Net-(U2-Pad11) -> unconnected-(U2-Pad11)
- U2 pad 9: Net-(U2-Pad9) -> unconnected-(U2-Pad9)
- U4 pad 7: Net-(U4-Pad7) -> unconnected-(U4-Pad7)
- U5 pad 1: Net-(U5-Pad1) -> unconnected-(U5-Pad1)
- U6 pad 20: Net-(U6-Pad20) -> unconnected-(U6-Pad20)
- U8 pad 19: Net-(U8-Pad19) -> unconnected-(U8-Pad19)
- U8 pad 2: Net-(U8-Pad2) -> unconnected-(U8-Pad2)
- U8 pad 22: Net-(U8-Pad22) -> unconnected-(U8-Pad22)
- U8 pad 23: Net-(U8-Pad23) -> unconnected-(U8-Pad23)
- U8 pad 24: Net-(U8-Pad24) -> unconnected-(U8-Pad24)
- U8 pad 5: Net-(U8-Pad5) -> unconnected-(U8-Pad5)
- U8 pad 6: Net-(U8-Pad6) -> unconnected-(U8-Pad6)
- U8 pad 7: Net-(U8-Pad7) -> unconnected-(U8-Pad7)
- U8 pad 8: Net-(U8-Pad8) -> unconnected-(U8-Pad8)
- U9 pad 1: Net-(U9-Pad1) -> unconnected-(U9-Pad1)
- U9 pad 10: Net-(U9-Pad10) -> unconnected-(U9-Pad10)
- U9 pad 11: Net-(U9-Pad11) -> unconnected-(U9-Pad11)
- U9 pad 12: Net-(U9-Pad12) -> unconnected-(U9-Pad12)
- U9 pad 13: Net-(U9-Pad13) -> unconnected-(U9-Pad13)
- U9 pad 14: Net-(U9-Pad14) -> unconnected-(U9-Pad14)
- U9 pad 15: Net-(U9-Pad15) -> unconnected-(U9-Pad15)
- U9 pad 16: Net-(U9-Pad16) -> unconnected-(U9-Pad16)
- U9 pad 17: Net-(U9-Pad17) -> unconnected-(U9-Pad17)
- U9 pad 18: Net-(U9-Pad18) -> unconnected-(U9-Pad18)
- U9 pad 19: Net-(U9-Pad19) -> unconnected-(U9-Pad19)
- U9 pad 22: Net-(U9-Pad22) -> unconnected-(U9-Pad22)
- U9 pad 24: Net-(U9-Pad24) -> unconnected-(U9-Pad24)
