File: Mainboard/AIO438.kicad_pcb (KiCad board)
At the start: 4 copper layers, 121 x 60 mm, 164 parts, among them J1 JST-PH 01x03, J10 U.FL, J11 JST-PH 01x02, J2 JST-PH 01x10, J3 PinHeader 02x03, J4 5mm screwterminal 01x12, J5 JST-PH 01x02, J6 JST-PH 01x02, J7 JST-PH 01x08, J8 USB-C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

Commit message: Do board setup and clear any DRC errors
Only DRC error left remaining is related to the antenna.
Library setup is still broken right now.
Parts:
- AE1: footprint RF_Antenna:Texas_SWRA117D_2.4GHz_Left -> ZOUDIO-footprints:Texas_SWRA117D_2.4GHz_Left
Routing:
- net GND: track 40.5 -> 35.3 mm
- net Net-(C28-Pad1): track 11.3 -> 7.45 mm
- net /Microcontroller/I2C_SDA: track 111.4 -> 108.8 mm
- net /Microcontroller/RESET: track 112.2 -> 110.1 mm
- net Net-(C26-Pad1): track 18.5 -> 16.4 mm
- net Net-(C9-Pad1): track 8.68 -> 7.28 mm
- net Net-(C27-Pad1): track 8.90 -> 7.53 mm
- net Net-(C10-Pad1): track 8.61 -> 7.24 mm
- net VDD: track 37.2 -> 36.1 mm
- net Net-(U8-Pad4): track 4.14 -> 3.45 mm
- net +3V3: track 36.3 -> 35.6 mm
- net /Power/3V3_buck: track 26.4 -> 25.8 mm
- net /Bluetooth/MIC1_P: track 144.1 -> 143.5 mm
