File: Mainboard/Bluetooth.kicad_sch (KiCad schematic)
At the start: 22 parts, among them J10 U.FL, J11 JST-PH 01x02, U10 BTM331

Commit message: Do board setup and clear any DRC errors
Only DRC error left remaining is related to the antenna.
Library setup is still broken right now.
Parts:
- AE1: footprint RF_Antenna:Texas_SWRA117D_2.4GHz_Left -> ZOUDIO-footprints:Texas_SWRA117D_2.4GHz_Left
Changed lines of the file:
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@@
       (effects (font (size 1.27 1.27)) (justify right))
     )
-    (property "Footprint" "RF_Antenna:Texas_SWRA117D_2.4GHz_Left" (id 2) (at 123.19 52.07 0)
+    (property "Footprint" "ZOUDIO-footprints:Texas_SWRA117D_2.4GHz_Left" (id 2) (at 123.19 52.07 0)
       (effects (font (size 1.27 1.27)) hide)
     )
