File: PCB/Mainboard/Amplifiers.kicad_sch (KiCad schematic)
At the start: 4 parts, among them J1 JST-PH 01x03, J4 5mm screwterminal 01x12

Commit message: Update schematic and lay-out
- Swap out CP2102N, ATmega328PB and CP with new Kicad 6 symbol
- Correct all links to point to new zoudio_symbols and zoudio_footprint libraries
- Lay-out updated, only antenna is left to update.
Parts:
- removed C1: 1000u, ZOUDIO-footprints:Cap_Rad_D10_P5_horizontal, symbol Device:CP
- added C1: 1000u, zoudio_footprints:Cap_Rad_D10_P5_horizontal, symbol Device:C_Polarized
- J4: footprint ZOUDIO-footprints:Multicomp_12P_5mm -> zoudio_footprints:Multicomp_12P_5mm
Connections:
- net GND: now also C1.2
- net VDD: now also C1.1
Changed lines of the file:
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@@
     (pin "1")
-  )
-  (symbol (lib_id "Device:CP") (at 147.32 139.7 0) (unit 1)
-    (in_bom yes) (on_board yes)
-    (property "Reference" "C1" (id 0) (at 149.86 139.7 0)
-      (effects (font (size 1.27 1.27)) (justify left))
-    )
-    (property "Value" "1000u" (id 1) (at 148.59 142.24 0)
-      (effects (font (size 1.27 1.27)) (justify left))
-    )
-    (property "Footprint" "ZOUDIO-footprints:Cap_Rad_D10_P5_horizontal" (id 2) (at 148.2852 143.51 0)
-      (effects (font (size 1.27 1.27)) hide)
-    )
-    (property "Datasheet" "~" (id 3) (at 147.32 139.7 0)
-      (effects (font (size 1.27 1.27)) hide)
-    )
-    (property "Manufacturer" "Nichicon" (id 4) (at 147.32 139.7 0)
-      (effects (font (size 1.27 1.27)) hide)
-    )
-    (property "Partnumber" "UHV1V102MHD" (id 5) (at 147.32 139.7 0)
-      (effects (font (size 1.27 1.27)) hide)
-    )
-    (pin "1")
-    (pin "2")
   )
   (symbol (lib_id "power:GND") (at 147.32 144.78 0) (mirror y) (unit 1)
@@
     (property "Reference" "J4" (id 0) (at 193.04 83.82 0))
     (property "Value" "5mm screwterminal 01x12" (id 1) (at 203.2 86.36 0))
-    (property "Footprint" "ZOUDIO-footprints:Multicomp_12P_5mm" (id 2) (at 187.96 88.9 0)
+    (property "Footprint" "zoudio_footprints:Multicomp_12P_5mm" (id 2) (at 187.96 88.9 0)
       (effects (font (size 1.27 1.27)) hide)
     )
@@
     (pin "1")
   )
+  (symbol (lib_id "Device:C_Polarized") (at 147.32 139.7 0) (unit 1)
+    (in_bom yes) (on_board yes) (fields_autoplaced)
+    (property "Reference" "C1" (id 0) (at 151.13 137.5409 0)
+      (effects (font (size 1.27 1.27)) (justify left))
+    )
+    (property "Value" "1000u" (id 1) (at 151.13 140.0809 0)
+      (effects (font (size 1.27 1.27)) (justify left))
+    )
+    (property "Footprint" "zoudio_footprints:Cap_Rad_D10_P5_horizontal" (id 2) (at 148.2852 143.51 0)
+      (effects (font (size 1.27 1.27)) hide)
+    )
+    (property "Datasheet" "~" (id 3) (at 147.32 139.7 0)
+      (effects (font (size 1.27 1.27)) hide)
+    )
+    (property "Manufacturer" "Nichicon" (id 4) (at 147.32 139.7 0)
+      (effects (font (size 1.27 1.27)) hide)
+    )
+    (property "Partnumber" "UHV1V102MHD" (id 5) (at 147.32 139.7 0)
+      (effects (font (size 1.27 1.27)) hide)
+    )
+    (pin "1")
+    (pin "2")
+  )
   (sheet (at 137.16 91.44) (size 21.59 27.94) (fields_autoplaced)
