File: PCB/Mainboard-TPCB/AIO438.kicad_sch (KiCad schematic)
At the start: 3 parts

Commit message: TPCB files V2
Parts:
- removed R1, R2: 0R, Resistor_SMD:R_0603_1608Metric, symbol Device:R_Small
- removed TP6: test, TestPoint:TestPoint_Pad_D1.0mm, symbol Connector:TestPoint
- added J10: PJ-324M, zoudio_footprints:PJ-324M, symbol zoudio_symbols:PJ-324M
Connections:
- net Mainboard (DUT)/AUX_GND: now also J10.S
- net Mainboard (DUT)/AUX_L: now also J10.T
- net Mainboard (DUT)/AUX_R: now also J10.R
- no-connect marks 0 -> 2
Other:
- sheet Dummy load A renamed Power IO
- removed sheet Dummy load B
- removed sheet Dummy load C
- removed sheet Dummy load D
- removed sheet Load switch
- removed sheet Power
- sheet MTM ports: added none; removed A3, D13, D14, D9
- sheet Power IO ports: added A+, A-, B+, B-, C+, C-, D+, D-, Vin; removed CH+, CH-
- note removed: "24V input 24V to 9V"
