File: PCB/Mainboard-TPCB/dummy_load.kicad_sch (KiCad schematic)
At the start: 4 parts, among them J23 Conn_Coaxial, J24 Conn_Coaxial

Commit message: TPCB files V2
Parts:
- removed J23, J24: Conn_Coaxial, Connector_Coaxial:SMA_Molex_73251-2200_Horizontal, symbol Connector:Conn_Coaxial
- added J9: 5mm screwterminal 01x12, Connector_Phoenix_MSTB:PhoenixContact_MSTBA_2,5_12-G-5,08_1x12_P5.08mm_Horizontal, symbol Connector_Generic:Conn_01x12
- added R10, R3, R4, R5, R8, R9: 2R, Package_TO_SOT_SMD:TO-252-2, symbol Device:R_Potentiometer
- renumbered R14 to R1, R15 to R2
Connections:
- net GND: now also J9.1 (Pin_1), J9.4 (Pin_4), R10.2, R3.2, R4.2, R5.2, R8.2, R9.2
- net CH+ renamed A+
- net A+: now also J9.5 (Pin_5)
- net CH- renamed A-
- net A-: now also J9.6 (Pin_6)
- new net: R3.3, R4.1
- new net: R10.1, R9.3
- new net: R5.3, R8.1
- new net B+: J9.8 (Pin_8), R4.3
- new net B-: J9.7 (Pin_7), R3.1
- new net C+: J9.9 (Pin_9), R5.1
- new net C-: J9.10 (Pin_10), R8.3
- new net D+: J9.12 (Pin_12), R10.3
- new net D-: J9.11 (Pin_11), R9.1
- new net Vin: J9.2 (Pin_2), J9.3 (Pin_3)
Other:
- note removed: "Pin 2 = heatsink"
- moved on the sheet: R1, R2
