File: PCB/Mainboard-TPCB/mainboard.kicad_sch (KiCad schematic)
At the start: 13 parts, among them J1 JST-PH 01x03, J11 JST-PH 01x02, J2 JST-PH 01x10, J3 PinHeader 02x03, J4 5mm screwterminal 01x12, J5 JST-PH 01x02, J6 JST-PH 01x02, J7 JST-PH 01x08

Commit message: TPCB files V2
Parts:
- R17, R6: Manufacturer Yageo -> (none); Partnumber RC0603FR-071KL -> (none)
- R7: Manufacturer Yageo -> (none); Partnumber RC0603FR-0710KL -> (none)
Other:
- note added: "Vin applied to both PSU and CHG inputs"
Changed lines of the file:
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@@
+    (effects (font (size 1.27 1.27)) (justify right bottom))
+  )
+  (text "Vin applied to both \nPSU and CHG inputs" (at 196.85 101.6 180)
     (effects (font (size 1.27 1.27)) (justify right bottom))
   )
@@
       (effects (font (size 1.27 1.27)) hide)
     )
-    (property "Manufacturer" "Yageo" (id 4) (at 113.03 133.35 0)
-      (effects (font (size 1.27 1.27)) hide)
-    )
-    (property "Partnumber" "RC0603FR-071KL" (id 5) (at 113.03 133.35 0)
+    (property "Manufacturer" "" (id 4) (at 113.03 133.35 0)
+      (effects (font (size 1.27 1.27)) hide)
+    )
+    (property "Partnumber" "" (id 5) (at 113.03 133.35 0)
       (effects (font (size 1.27 1.27)) hide)
     )
@@
       (effects (font (size 1.27 1.27)) hide)
     )
-    (property "Manufacturer" "Yageo" (id 4) (at 115.57 151.13 0)
-      (effects (font (size 1.27 1.27)) hide)
-    )
-    (property "Partnumber" "RC0603FR-0710KL" (id 5) (at 115.57 151.13 0)
+    (property "Manufacturer" "" (id 4) (at 115.57 151.13 0)
+      (effects (font (size 1.27 1.27)) hide)
+    )
+    (property "Partnumber" "" (id 5) (at 115.57 151.13 0)
       (effects (font (size 1.27 1.27)) hide)
     )
@@
       (effects (font (size 1.27 1.27)) hide)
     )
-    (property "Manufacturer" "Yageo" (id 4) (at 175.26 44.45 0)
-      (effects (font (size 1.27 1.27)) hide)
-    )
-    (property "Partnumber" "RC0603FR-071KL" (id 5) (at 175.26 44.45 0)
-      (effects (font (size 1.27 1.27)) hide)
-    )
+    (property "Manufacturer" "" (id 4) (at 175.26 44.45 0)
+      (effects (font (size 1.27 1.27)) hide)
+    )
+    (property "Partnumber" "" (id 5) (at 175.26 44.45 0)
+      (effects (font (size 1.27 1.27)) hide)
+    )
