File: PCB/Mainboard-TPCB/misc.kicad_sch (KiCad schematic)
At the start: 5 parts

Commit message: TPCB files V2
Parts:
- LOGO1: footprint zoudio_footprints:ZOUDIO25mm_mask -> zoudio_footprints:ZOUDIO25mm
Changed lines of the file:
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@@
     )
     (property "Value" "ZOUDIO" (id 1) (at 149.86 101.6 0))
-    (property "Footprint" "zoudio_footprints:ZOUDIO25mm_mask" (id 2) (at 149.86 95.25 0)
+    (property "Footprint" "zoudio_footprints:ZOUDIO25mm" (id 2) (at 149.86 95.25 0)
       (effects (font (size 1.27 1.27)) hide)
     )
